File: hw_v1/hw_v1.kicad_pcb (KiCad board)
At the start: 0 parts

Commit message: wip pcb layout
Parts:
- added A1: Pololu_Breakout_DRV8825, Module:Pololu_Breakout-16_15.2x20.3mm, F.Cu at (150.8, 130.7)
- added BT1: Battery_Cell, Connector_JST:JST_EH_B2B-EH-A_1x02_P2.50mm_Vertical, F.Cu at (204.9, 96.6)
- added C1: 0.01uF, Capacitor_SMD:C_0805_2012Metric, F.Cu at (221.9, 64.4)
- added C11: 100nF, Capacitor_SMD:C_0805_2012Metric, F.Cu at (176.5, 106.6)
- added C12: 100nF, Capacitor_SMD:C_0805_2012Metric, F.Cu at (176.5, 109.6)
- added C13: 100nF, Capacitor_SMD:C_0805_2012Metric, F.Cu at (176.5, 112.6)
- added C14: 100nF, Capacitor_SMD:C_0805_2012Metric, F.Cu at (116.3, 63.8)
- added C15: 47nF, Capacitor_SMD:C_0603_1608Metric, F.Cu at (107.0, 64.0)
- added C16: 0.22uF, Capacitor_SMD:C_0603_1608Metric, F.Cu at (180.8, 124.1)
- added C17: 0.22uF, Capacitor_SMD:C_0603_1608Metric, F.Cu at (180.8, 126.6)
- added C18: 0.22uF, Capacitor_SMD:C_0603_1608Metric, F.Cu at (180.8, 129.1)
- added C19: 0.1uF, Capacitor_SMD:C_0805_2012Metric, F.Cu at (234.9, 131.5)
- added C2: 0.01uF, Capacitor_SMD:C_0805_2012Metric, F.Cu at (221.9, 67.4)
- added C20: 0.1uF, Capacitor_SMD:C_0805_2012Metric, F.Cu at (234.9, 134.5)
- added C21: 100nF, Capacitor_SMD:C_0805_2012Metric, F.Cu at (176.5, 115.6)
- added C22: 100nF, Capacitor_SMD:C_0805_2012Metric, F.Cu at (176.5, 118.7)
- added C23: 100nF, Capacitor_SMD:C_0805_2012Metric, F.Cu at (176.5, 121.7)
- added C24: 0.22uF, Capacitor_SMD:C_0603_1608Metric, F.Cu at (180.8, 131.6)
- added C25: 0.1uF, Capacitor_SMD:C_0805_2012Metric, F.Cu at (234.9, 137.5)
- added C26: 2.2uF, Capacitor_SMD:C_0805_2012Metric, F.Cu at (195.0, 64.4)
- added C27: 0.22uF, Capacitor_SMD:C_0603_1608Metric, F.Cu at (180.8, 134.1)
- added C28: 0.22uF, Capacitor_SMD:C_0603_1608Metric, F.Cu at (180.8, 136.6)
- added C29: 2.2uF, Capacitor_SMD:C_0805_2012Metric, F.Cu at (195.0, 67.4)
- added C3: 0.01uF, Capacitor_SMD:C_0805_2012Metric, F.Cu at (221.9, 70.4)
- added C30: 100nF, Capacitor_SMD:C_0805_2012Metric, F.Cu at (195.0, 70.4)
- added C31: 100nF, Capacitor_SMD:C_0805_2012Metric, F.Cu at (195.0, 73.4)
- added C32: 100nF, Capacitor_SMD:C_0805_2012Metric, F.Cu at (199.5, 64.4)
- added C33: 100nF, Capacitor_SMD:C_0805_2012Metric, F.Cu at (199.5, 67.4)
- added C34: 1uF, Capacitor_SMD:C_0805_2012Metric, F.Cu at (199.5, 70.4)
- added C35: 100nF, Capacitor_SMD:C_0805_2012Metric, F.Cu at (199.5, 73.4)
- added C36: 100nF, Capacitor_SMD:C_0805_2012Metric, F.Cu at (203.9, 64.4)
- added C37: 100nF, Capacitor_SMD:C_0805_2012Metric, F.Cu at (203.9, 67.4)
- added C38: 4.7uF, Capacitor_SMD:C_0805_2012Metric, F.Cu at (203.9, 70.4)
- added C39: 100nF, Capacitor_SMD:C_0805_2012Metric, F.Cu at (203.9, 73.4)
- added C4: 0.01uF, Capacitor_SMD:C_0805_2012Metric, F.Cu at (221.9, 73.4)
- added C40: 6.8pF, Capacitor_SMD:C_0805_2012Metric, F.Cu at (208.4, 64.4)
- added C41: 6.8pF, Capacitor_SMD:C_0805_2012Metric, F.Cu at (208.4, 67.4)
- added C42: 15pF, Capacitor_SMD:C_0805_2012Metric, F.Cu at (208.4, 70.4)
- added C43: 15pF, Capacitor_SMD:C_0805_2012Metric, F.Cu at (208.4, 73.4)
- added C44: 1u, Capacitor_SMD:C_0402_1005Metric, F.Cu at (188.3, 91.9)
- added C45: 1u, Capacitor_SMD:C_0402_1005Metric, F.Cu at (188.3, 93.8)
- added C46: 100n, Capacitor_SMD:C_0402_1005Metric, F.Cu at (188.3, 95.8)
- added C47: 100nF, Capacitor_SMD:C_0805_2012Metric, F.Cu at (114.8, 104.1)
- added C48: 47nF, Capacitor_SMD:C_0603_1608Metric, F.Cu at (119.7, 64.0)
- added C49: 100nF, Capacitor_SMD:C_0805_2012Metric, F.Cu at (128.9, 63.8)
- added C5: 0.01uF, Capacitor_SMD:C_0805_2012Metric, F.Cu at (221.9, 76.4)
- added C50: 100nF, Capacitor_SMD:C_0805_2012Metric, F.Cu at (114.8, 107.1)
- added C51: 0.1uF, Capacitor_SMD:C_0805_2012Metric, F.Cu at (79.6, 60.3)
- added C52: 0.1uF, Capacitor_SMD:C_0805_2012Metric, F.Cu at (95.0, 56.5)
- added C53: 0.1uF, Capacitor_SMD:C_0805_2012Metric, F.Cu at (79.7, 56.4)
- added C54: 10nF, Capacitor_SMD:C_0805_2012Metric, F.Cu at (100.4, 58.9)
- added C55: 100uF ±20% 35V, Capacitor_SMD:CP_Elec_6.3x7.7, F.Cu at (91.9, 62.6)
- added C6: 0.01uF, Capacitor_SMD:C_0805_2012Metric, F.Cu at (221.9, 79.4)
- added C7: 0.01uF, Capacitor_SMD:C_0805_2012Metric, F.Cu at (221.9, 82.4)
- added C8: 4700pF, Capacitor_SMD:C_0805_2012Metric, F.Cu at (221.9, 85.4)
- added D1: LED, LED_SMD:LED_0805_2012Metric, F.Cu at (244.6, 91.6)
- added D10: LED, LED_SMD:LED_0805_2012Metric, F.Cu at (244.6, 109.9)
- added D11: D, Diode_SMD:D_SOD-323_HandSoldering, F.Cu at (257.8, 100.4)
- added D12: LED, LED_SMD:LED_0805_2012Metric, F.Cu at (244.6, 112.9)
- added D16: 1N4148, Diode_SMD:D_SOD-523, F.Cu at (222.8, 133.7)
- added D17: 1N4148, Diode_SMD:D_SOD-523, F.Cu at (222.8, 136.2)
- added D18: 1N4148, Diode_SMD:D_SOD-523, F.Cu at (188.6, 101.6)
- added D19: 1N5819WS, Diode_SMD:D_SOD-323_HandSoldering, F.Cu at (209.5, 101.3)
- added D2: LED, LED_SMD:LED_0805_2012Metric, F.Cu at (244.6, 94.7)
- added D20: LED, LED_SMD:LED_0805_2012Metric, F.Cu at (176.6, 82.9)
- added D21: LED, LED_SMD:LED_0805_2012Metric, F.Cu at (176.6, 85.9)
- added D22: LED, LED_SMD:LED_0805_2012Metric, F.Cu at (176.6, 88.9)
- added D23: LED, LED_SMD:LED_0805_2012Metric, F.Cu at (176.6, 92.0)
- added D24: LED, LED_SMD:LED_0805_2012Metric, F.Cu at (176.6, 95.0)
- added D25: LED, LED_SMD:LED_0805_2012Metric, F.Cu at (176.6, 98.1)
- added D26: LED, LED_SMD:LED_0805_2012Metric, F.Cu at (176.6, 101.1)
- added D27: 3.1v, Diode_SMD:D_SOD-323, F.Cu at (232.4, 91.6)
- added D28: MM3Z24VT1G, Diode_SMD:D_SOD-323, F.Cu at (256.1, 136.4)
- added D29: D, Diode_SMD:D_SOD-123F, F.Cu at (241.9, 126.0)
- added D3: D, Diode_SMD:D_SOD-323_HandSoldering, F.Cu at (257.8, 91.6)
- added D30: D, Diode_SMD:D_SOD-123F, F.Cu at (241.9, 129.3)
- added D31: 3.1v, Diode_SMD:D_SOD-323, F.Cu at (232.4, 94.5)
- added D32: 3.1v, Diode_SMD:D_SOD-323, F.Cu at (232.4, 97.5)
- added D33: 3.1v, Diode_SMD:D_SOD-323, F.Cu at (232.4, 100.4)
- added D34: 3.1v, Diode_SMD:D_SOD-323, F.Cu at (232.4, 103.4)
- added D35: SM6T33A, Diode_SMD:D_SMB, F.Cu at (70.9, 85.6)
- added D4: LED, LED_SMD:LED_0805_2012Metric, F.Cu at (244.6, 97.7)
- added D5: LED, LED_SMD:LED_0805_2012Metric, F.Cu at (244.6, 100.7)
- added D6: D, Diode_SMD:D_SOD-323_HandSoldering, F.Cu at (257.8, 94.5)
- added D7: LED, LED_SMD:LED_0805_2012Metric, F.Cu at (244.6, 103.8)
- added D8: D, Diode_SMD:D_SOD-323_HandSoldering, F.Cu at (257.8, 97.5)
- added D9: LED, LED_SMD:LED_0805_2012Metric, F.Cu at (244.6, 106.8)
- added F1: Polyfuse, Fuse:Fuse_1812_4532Metric, F.Cu at (217.5, 135.0)
- added J10: Conn_01x01, TestPoint:TestPoint_THTPad_2.0x2.0mm_Drill1.0mm, F.Cu at (241.1, 133.0)
- added J11: Conn_01x01, TestPoint:TestPoint_THTPad_2.0x2.0mm_Drill1.0mm, F.Cu at (241.1, 137.1)
- added J12: Delphi_Sicma_24, uEFI_v5:Delphi_Sicma_24_Grey, F.Cu at (50.0, 128.7)
- added J13: Delphi_Sicma_24, uEFI_v5:Delphi_Sicma_24_Black, F.Cu at (50.0, 75.3)
- added J14: Conn_01x04, Connector_PinHeader_2.54mm:PinHeader_1x04_P2.54mm_Vertical, F.Cu at (136.1, 61.1)
- added J2: Conn_01x05, Connector_PinHeader_2.54mm:PinHeader_1x05_P2.54mm_Vertical, F.Cu at (216.4, 120.0)
- added J3: Conn_01x05, Connector_PinHeader_2.54mm:PinHeader_1x05_P2.54mm_Vertical, F.Cu at (221.0, 120.0)
- added J4: Conn_01x05, Connector_PinHeader_2.54mm:PinHeader_1x05_P2.54mm_Vertical, F.Cu at (225.7, 120.0)
- added J5: Conn_01x03, Connector_PinHeader_2.54mm:PinHeader_1x03_P2.54mm_Vertical, F.Cu at (230.3, 132.3)
- added J6: Conn_01x04, Connector_PinHeader_2.54mm:PinHeader_1x04_P2.54mm_Vertical, F.Cu at (230.3, 120.0)
- added J8: USB_B, Connector_USB:USB_Mini-B_Tensility_54-00023_Vertical, F.Cu at (149.4, 81.7)
- added J9: Tag connect, Connector:Tag-Connect_TC2030-IDC-FP_2x03_P1.27mm_Vertical, F.Cu at (149.7, 69.3)
- added JP1: Jumper_3_Bridged12, Jumper:SolderJumper-3_P1.3mm_Bridged12_Pad1.0x1.5mm, F.Cu at (231.8, 79.7)
- added JP10: SolderJumper_3_Bridged12, Jumper:SolderJumper-3_P1.3mm_Bridged2Bar12_Pad1.0x1.5mm, F.Cu at (141.9, 58.2)
- added JP11: Jumper_2_Open, Jumper:SolderJumper-2_P1.3mm_Open_RoundedPad1.0x1.5mm, F.Cu at (231.2, 63.6)
- added JP12: Jumper_2_Open, Jumper:SolderJumper-2_P1.3mm_Open_RoundedPad1.0x1.5mm, F.Cu at (231.2, 67.2)
- added JP2: Jumper_3_Bridged12, Jumper:SolderJumper-3_P1.3mm_Bridged12_Pad1.0x1.5mm, F.Cu at (231.8, 83.5)
- added JP3: SolderJumper_2_Open, Jumper:SolderJumper-2_P1.3mm_Open_RoundedPad1.0x1.5mm, F.Cu at (239.0, 64.6)
- added JP4: SolderJumper_2_Open, Jumper:SolderJumper-2_P1.3mm_Open_RoundedPad1.0x1.5mm, F.Cu at (239.0, 68.2)
- added JP5: Jumper_2_Open, Jumper:SolderJumper-2_P1.3mm_Bridged2Bar_Pad1.0x1.5mm, F.Cu at (189.0, 98.6)
- added JP6: Jumper_2_Open, Jumper:SolderJumper-2_P1.3mm_Open_Pad1.0x1.5mm, F.Cu at (256.1, 126.1)
- added JP7: Jumper_2_Open, Jumper:SolderJumper-2_P1.3mm_Open_Pad1.0x1.5mm, F.Cu at (256.1, 129.6)
- added JP8: Jumper_2_Open, Jumper:SolderJumper-2_P1.3mm_Open_Pad1.0x1.5mm, F.Cu at (256.1, 133.2)
- added JP9: SolderJumper_3_Bridged12, Jumper:SolderJumper-3_P1.3mm_Bridged2Bar12_Pad1.0x1.5mm, F.Cu at (138.1, 58.2)
- added Q1: AO3400A, Package_TO_SOT_SMD:SOT-23, F.Cu at (226.6, 80.1)
- added Q2: AO3400A, Package_TO_SOT_SMD:SOT-23, F.Cu at (226.6, 84.6)
- added Q3: FDS6890A, Package_SO:SOP-8_3.9x4.9mm_P1.27mm, F.Cu at (83.6, 58.4)
- added Q5: SS8050, Package_TO_SOT_SMD:SOT-23, F.Cu at (247.1, 126.5)
- added Q6: AO3400A, Package_TO_SOT_SMD:SOT-23, F.Cu at (247.1, 131.0)
- added R1: 10k, Resistor_SMD:R_0805_2012Metric, F.Cu at (257.3, 104.5)
- added R10: 10k, Resistor_SMD:R_0603_1608Metric, F.Cu at (236.7, 84.2)
- added R11: 10k, Resistor_SMD:R_0603_1608Metric, F.Cu at (236.7, 86.7)
- added R12: 470R, Resistor_SMD:R_0805_2012Metric, F.Cu at (234.9, 119.2)
- added R13: 470R, Resistor_SMD:R_0805_2012Metric, F.Cu at (234.9, 122.1)
- added R14: 2.49k +-1%, Resistor_SMD:R_0603_1608Metric, F.Cu at (184.8, 124.1)
- added R15: 2.49k +-1%, Resistor_SMD:R_0603_1608Metric, F.Cu at (184.8, 126.6)
- added R16: 1k, Resistor_SMD:R_0805_2012Metric, F.Cu at (234.9, 125.1)
- added R17: 180k, Resistor_SMD:R_0805_2012Metric, F.Cu at (181.0, 106.6)
- added R18: 470R, Resistor_SMD:R_0603_1608Metric, F.Cu at (184.8, 129.1)
- added R19: 470R, Resistor_SMD:R_0603_1608Metric, F.Cu at (184.8, 131.6)
- added R2: 10K 1/2W, Resistor_SMD:R_1210_3225Metric, F.Cu at (216.9, 65.0)
- added R20: 470R, Resistor_SMD:R_0603_1608Metric, F.Cu at (184.8, 134.1)
- added R21: 604R, Resistor_SMD:R_0805_2012Metric, F.Cu at (181.0, 109.5)
- added R22: 3.88k, Resistor_SMD:R_0603_1608Metric, F.Cu at (184.8, 136.6)
- added R23: 348k, Resistor_SMD:R_0805_2012Metric, F.Cu at (181.0, 112.5)
- added R24: 180k, Resistor_SMD:R_0805_2012Metric, F.Cu at (181.0, 115.4)
- added R25: 2.49k +-1%, Resistor_SMD:R_0603_1608Metric, F.Cu at (188.8, 124.1)
- added R26: 348k, Resistor_SMD:R_0805_2012Metric, F.Cu at (181.0, 118.4)
- added R27: 10k, Resistor_SMD:R_0603_1608Metric, F.Cu at (180.8, 82.6)
- added R28: 470R, Resistor_SMD:R_0603_1608Metric, F.Cu at (188.8, 126.6)
- added R29: 470R, Resistor_SMD:R_0603_1608Metric, F.Cu at (188.8, 129.1)
- added R3: 10K 1/2W, Resistor_SMD:R_1210_3225Metric, F.Cu at (216.9, 69.2)
- added R30: 470R, Resistor_SMD:R_0603_1608Metric, F.Cu at (188.8, 131.6)
- added R31: 120R, Resistor_SMD:R_1206_3216Metric, F.Cu at (204.2, 101.5)
- added R32: 4.7k, Resistor_SMD:R_0603_1608Metric, F.Cu at (180.8, 85.1)
- added R33: 180k, Resistor_SMD:R_0805_2012Metric, F.Cu at (181.0, 121.3)
- added R34: 4.7k, Resistor_SMD:R_0603_1608Metric, F.Cu at (180.8, 87.6)
- added R35: 180k, Resistor_SMD:R_0805_2012Metric, F.Cu at (185.4, 106.6)
- added R36: 180k, Resistor_SMD:R_0805_2012Metric, F.Cu at (185.4, 109.5)
- added R37: 4.7k, Resistor_SMD:R_0603_1608Metric, F.Cu at (180.8, 90.1)
- added R38: 4.7k, Resistor_SMD:R_0603_1608Metric, F.Cu at (180.8, 92.6)
- added R39: 348k, Resistor_SMD:R_0805_2012Metric, F.Cu at (185.4, 112.5)
- added R4: 10K 1/2W, Resistor_SMD:R_1210_3225Metric, F.Cu at (216.9, 73.4)
- added R40: 348k, Resistor_SMD:R_0805_2012Metric, F.Cu at (185.4, 115.4)
- added R41: 348k, Resistor_SMD:R_0805_2012Metric, F.Cu at (185.4, 118.4)
- added R42: 4.7k, Resistor_SMD:R_0603_1608Metric, F.Cu at (180.8, 95.1)
- added R43: 4.7k, Resistor_SMD:R_0603_1608Metric, F.Cu at (180.8, 97.7)
- added R44: 4.7k, Resistor_SMD:R_0603_1608Metric, F.Cu at (180.8, 100.2)
- added R45: 180k, Resistor_SMD:R_0805_2012Metric, F.Cu at (185.4, 121.3)
- added R46: 180k, Resistor_SMD:R_0805_2012Metric, F.Cu at (189.8, 106.6)
- added R47: 180k, Resistor_SMD:R_0805_2012Metric, F.Cu at (189.8, 109.5)
- added R48: 1k, Resistor_SMD:R_0603_1608Metric, F.Cu at (228.2, 101.4)
- added R49: 1k, Resistor_SMD:R_0603_1608Metric, F.Cu at (228.2, 103.9)
- added R5: 10K 1/2W, Resistor_SMD:R_1210_3225Metric, F.Cu at (216.9, 77.6)
- added R50: 348k, Resistor_SMD:R_0805_2012Metric, F.Cu at (189.8, 112.5)
- added R51: 348k, Resistor_SMD:R_0805_2012Metric, F.Cu at (189.8, 115.4)
- added R52: 348k, Resistor_SMD:R_0805_2012Metric, F.Cu at (189.8, 118.4)
- added R53: 1k, Resistor_SMD:R_0603_1608Metric, F.Cu at (246.6, 134.5)
- added R54: 100k, Resistor_SMD:R_0603_1608Metric, F.Cu at (246.6, 137.0)
- added R55: 100k, Resistor_SMD:R_0805_2012Metric, F.Cu at (251.7, 125.8)
- added R56: 100k, Resistor_SMD:R_0805_2012Metric, F.Cu at (251.7, 128.7)
- added R57: 1k, Resistor_SMD:R_0805_2012Metric, F.Cu at (251.7, 131.7)
- added R58: 1k, Resistor_SMD:R_0805_2012Metric, F.Cu at (251.7, 134.6)
- added R59: 1k, Resistor_SMD:R_0603_1608Metric, F.Cu at (228.2, 106.4)
- added R6: 1k, Resistor_SMD:R_0603_1608Metric, F.Cu at (236.7, 79.2)
- added R60: 1k, Resistor_SMD:R_0603_1608Metric, F.Cu at (228.2, 108.9)
- added R61: 1k, Resistor_SMD:R_0603_1608Metric, F.Cu at (228.2, 111.4)
- added R62: 90k, Resistor_SMD:R_0603_1608Metric, F.Cu at (98.3, 56.3)
- added R63: 900R, Resistor_SMD:R_0603_1608Metric, F.Cu at (96.8, 56.3)
- added R64: 9.09k, Resistor_SMD:R_0603_1608Metric, F.Cu at (99.9, 56.3)
- added R65: 3.48k, Resistor_SMD:R_0603_1608Metric, F.Cu at (101.3, 56.3)
- added R66: 1k, Resistor_SMD:R_0603_1608Metric, F.Cu at (87.5, 57.1)
- added R67: 100R, Resistor_SMD:R_0603_1608Metric, F.Cu at (97.0, 59.0)
- added R7: 4.99K 1/2W, Resistor_SMD:R_1210_3225Metric, F.Cu at (216.9, 81.8)
- added R8: 4.99K 1/2W, Resistor_SMD:R_1210_3225Metric, F.Cu at (216.9, 86.0)
- added R9: 1k, Resistor_SMD:R_0603_1608Metric, F.Cu at (236.7, 81.7)
- added REF**: MountingHole_3.2mm_M3_ISO14580_Pad, MountingHole:MountingHole_3.2mm_M3_ISO14580_Pad, F.Cu at (74.6, 58.8)
- added REF**: MountingHole_3.2mm_M3_ISO14580_Pad, MountingHole:MountingHole_3.2mm_M3_ISO14580_Pad, F.Cu at (157.6, 145.8)
- added REF**: MountingHole_3.2mm_M3_ISO14580_Pad, MountingHole:MountingHole_3.2mm_M3_ISO14580_Pad, F.Cu at (157.6, 58.8)
- added REF**: MountingHole_3.2mm_M3_ISO14580_Pad, MountingHole:MountingHole_3.2mm_M3_ISO14580_Pad, F.Cu at (74.6, 145.8)
- added RN1: 1k, Resistor_SMD:R_Array_Convex_4x0603, F.Cu at (248.9, 105.4)
- added RN2: 1k, Resistor_SMD:R_Array_Convex_4x0603, F.Cu at (253.0, 105.4)
- added RN3: 47k, Resistor_SMD:R_Array_Convex_4x0603, F.Cu at (204.2, 83.7)
- added RN4: 47k, Resistor_SMD:R_Array_Convex_4x0603, F.Cu at (208.4, 83.7)
- added SW2: SW_Push, Button_Switch_SMD:SW_SPST_TL3342, F.Cu at (148.3, 101.2)
- added TP1: TestPoint, TestPoint:TestPoint_Pad_1.0x1.0mm, F.Cu at (234.1, 72.7)
- added TP10: TestPoint_Alt, TestPoint:TestPoint_THTPad_1.0x1.0mm_Drill0.5mm, F.Cu at (193.5, 121.1)
- added TP11: TestPoint_Alt, TestPoint:TestPoint_THTPad_1.0x1.0mm_Drill0.5mm, F.Cu at (196.6, 118.1)
- added TP12: TestPoint, TestPoint:TestPoint_Pad_1.0x1.0mm, F.Cu at (209.6, 76.4)
- added TP13: TestPoint, TestPoint:TestPoint_Pad_1.0x1.0mm, F.Cu at (209.6, 79.5)
- added TP14: TestPoint_Alt, TestPoint:TestPoint_THTPad_1.0x1.0mm_Drill0.5mm, F.Cu at (196.6, 121.1)
- added TP15: TestPoint_Alt, TestPoint:TestPoint_THTPad_1.0x1.0mm_Drill0.5mm, F.Cu at (199.6, 118.1)
- added TP16: TestPoint_Alt, TestPoint:TestPoint_THTPad_1.0x1.0mm_Drill0.5mm, F.Cu at (199.6, 121.1)
- added TP2: TestPoint, TestPoint:TestPoint_Pad_1.0x1.0mm, F.Cu at (234.1, 75.8)
- added TP3: TestPoint, TestPoint:TestPoint_Pad_1.0x1.0mm, F.Cu at (237.2, 72.7)
- added TP4: TestPoint, TestPoint:TestPoint_Pad_1.0x1.0mm, F.Cu at (237.2, 75.8)
- added TP5: TestPoint, TestPoint:TestPoint_Pad_1.0x1.0mm, F.Cu at (240.2, 72.7)
- added TP6: TestPoint, TestPoint:TestPoint_Pad_1.0x1.0mm, F.Cu at (240.2, 75.8)
- added TP7: BOOT0, TestPoint:TestPoint_Pad_D2.0mm, F.Cu at (184.8, 92.9)
- added TP8: BOOT1, TestPoint:TestPoint_Pad_D2.0mm, F.Cu at (184.8, 97.0)
- added TP9: TestPoint_Alt, TestPoint:TestPoint_THTPad_1.0x1.0mm_Drill0.5mm, F.Cu at (193.5, 118.1)
- added U1: MCZ33810EK, uEFI_v5:SOP65P1030X245-33N, F.Cu at (97.1, 128.0)
- added U10: BMP280, Package_LGA:Bosch_LGA-8_2x2.5mm_P0.65mm_ClockwisePinNumbering, F.Cu at (176.4, 125.0)
- added U11: L78M05ABDT-TR, Package_TO_SOT_SMD:TO-252-2, F.Cu at (111.4, 59.1)
- added U12: LM74800, uEFI_v5:LM74800, F.Cu at (91.2, 54.7)
- added U13: STM32F407VGTx, Package_QFP:LQFP-100_14x14mm_P0.5mm, F.Cu at (126.5, 86.0)
- added U14: TJA1051T-3, Package_SO:SOP-8_3.9x4.9mm_P1.27mm, F.Cu at (196.0, 98.4)
- added U15: 25LCxxx, Package_SO:SOIC-8_5.275x5.275mm_P1.27mm, F.Cu at (148.7, 94.3)
- added U16: REF3033, Package_TO_SOT_SMD:SOT-23, F.Cu at (205.6, 77.1)
- added U17: SRV05-4, Package_TO_SOT_SMD:SOT-23-6, F.Cu at (200.6, 77.1)
- added U18: VNLD5090, Package_SO:SOIC-8_3.9x4.9mm_P1.27mm, F.Cu at (252.1, 120.9)
- added U19: L78M05ABDT-TR, Package_TO_SOT_SMD:TO-252-2, F.Cu at (124.1, 59.1)
- added U2: TC4424A, Package_SO:SOIC-8_3.9x4.9mm_P1.27mm, F.Cu at (80.4, 125.1)
- added U21: ADXL343, Package_LGA:LGA-14_3x5mm_P0.8mm_LayoutBorder1x6y, F.Cu at (110.3, 105.9)
- added U3: TC4424A, Package_SO:SOIC-8_3.9x4.9mm_P1.27mm, F.Cu at (80.4, 131.5)
- added U4: MAX9926UAEE+, Package_SO:QSOP-16_3.9x4.9mm_P0.635mm, F.Cu at (228.4, 74.6)
- added U5: TPL7407LAPWR, Package_SO:TSSOP-16_4.4x5mm_P0.65mm, F.Cu at (243.5, 121.0)
- added U6: LMV324, Package_SO:TSSOP-14_4.4x5mm_P0.65mm, F.Cu at (195.2, 126.1)
- added U7: LMV324, Package_SO:TSSOP-14_4.4x5mm_P0.65mm, F.Cu at (195.2, 132.6)
- added U9: SP720ABTG, Package_SO:SOP-16_3.9x9.9mm_P1.27mm, F.Cu at (196.3, 110.8)
- added Y1: 32.768kHz, Crystal:Crystal_SMD_2012-2Pin_2.0x1.2mm, F.Cu at (184.6, 100.4)
- added Y2: 25MHz, Crystal:Crystal_SMD_3225-4Pin_3.2x2.5mm, F.Cu at (195.4, 77.1)
Routing:
- net +12VA: track 0.00 -> 58.8 mm
- net +12V: track 0.00 -> 53.1 mm, vias 0 -> 2
- net Net-(U12-OV): track 0.00 -> 16.8 mm, vias 0 -> 2
- net Net-(Q3B-G2): track 0.00 -> 16.0 mm
- net Net-(U12-SW): track 0.00 -> 12.5 mm, vias 0 -> 2
- net Net-(U12-C): track 0.00 -> 6.97 mm, vias 0 -> 2
- net Net-(C53-Pad2): track 0.00 -> 5.94 mm
- net +5C: track 0.00 -> 4.85 mm, vias 0 -> 1
- net +5V: track 0.00 -> 4.56 mm, vias 0 -> 1
- net Net-(U12-CAP): track 0.00 -> 2.59 mm
- net Net-(U12-EN/UVLO): track 0.00 -> 2.47 mm
- net Net-(C54-Pad2): track 0.00 -> 1.62 mm
- net Net-(R62-Pad1): track 0.00 -> 1.52 mm
- net /Connector/VBATT_MON: track 0.00 -> 1.52 mm
- net GND: track 0.00 -> 0.80 mm, vias 0 -> 1
Other:
- board outline added: 116.5 x 98 mm
- copper layers 0 -> 4
- board text added: "MCU +5V"
- board text added: "Sensors +5V"
- board text added: "surge protection"
