File: hw_v1/hw_v1.kicad_pcb (KiCad board)
At the start: 4 copper layers, 116.5 x 98 mm, 241 parts, among them J10 Conn_01x01, J11 Conn_01x01, J12 Delphi_Sicma_24, J13 Delphi_Sicma_24, J14 Conn_01x04, J15 Conn_01x03, J2 Conn_01x05, J3 Conn_01x05, J4 Conn_01x05, J5 Conn_01x03, J6 Conn_01x04, J7 104031-0811, J8 USB_B, J9 Tag connect, Q1 AO3400A, Q2 AO3400A, Q3 FDS6890A, Q5 SS8050, Q6 AO3400A, SW2 SW_Push, U1 MCZ33810EK, U10 BMP280, U11 L78M05ABDT-TR, U12 LM74800, U13 STM32F407VGTx, U14 TJA1051T-3, U15 25LCxxx, U16 REF3033, U17 SRV05-4, U18 VNLD5090, U19 L78M05ABDT-TR, U2 TC4424A, U21 ADXL343, U3 TC4424A, U4 MAX9926UAEE+, U5 TPL7407LAPWR, U6 LMV324, U7 LMV324, U8 AMS1117-3.3, U9 SP720ABTG, Y1 32.768kHz, Y2 25MHz

Commit message: update SD card holder to Molex 47352
Parts:
- removed J7: 104031-0811, Connector_Card:microSD_HC_Molex_104031-0811
- removed RN4: 47k, Resistor_SMD:R_Array_Convex_4x0603
- added J16: 47352-1001, uEFI_v5:MOLEX_47352-1001, F.Cu at (158.3, 81.5)
- added JP14: Jumper_2_Open, Jumper:SolderJumper-2_P1.3mm_Open_TrianglePad1.0x1.5mm, F.Cu at (80.8, 65.7)
- U15: value 25LCxxx -> 25Q16
- moved G*** 25.7 mm to (100.9, 76.3)
- moved C35 1.30 mm to (149.4, 81.8)
- moved RN3 1.11 mm to (148.7, 85.5)
Connections:
- net /SD_CLK renamed /SPI3_MOSI
- RN3 pad 1: unconnected-(RN3-R1.1-Pad1) -> /SD_CARD_DETECT
- RN3 pad 3: /SD_DAT0 -> /SPI3_MISO
- RN3 pad 4: /SD_DAT1 -> /SPI3_SCk
- U13 pad 65: /SD_DAT0 -> /SD_CS
- U13 pad 66: /SD_DAT1 -> /SD_CARD_DETECT
- U13 pad 78: /SD_DAT2 -> /SPI3_SCk
- U13 pad 79: /SD_DAT3 -> /SPI3_MISO
- U13 pad 97: /fuel_pump -> /fan1
- U13 pad 98: /fan1 -> /fuel_pump
Routing:
- net /SD_CD: track 48.0 -> 0.00 mm, vias 2 -> 0
- net /SD_CMD: track 40.8 -> 0.00 mm, vias 3 -> 0
- net /SD_DAT0: track 40.0 -> 0.00 mm, vias 2 -> 0
- net /SD_DAT2: track 39.8 -> 0.00 mm, vias 2 -> 0
- net /SD_CARD_DETECT: track 0.00 -> 39.6 mm, vias 0 -> 3
- net /SD_CS: track 0.00 -> 39.2 mm, vias 0 -> 2
- net /SD_DAT3: track 36.4 -> 0.00 mm, vias 2 -> 0
- net /SPI3_SCk: track 0.00 -> 34.1 mm
- net /SD_DAT1: track 33.7 -> 0.00 mm, vias 2 -> 0
- net /SPI3_MISO: track 0.00 -> 30.9 mm, vias 0 -> 2
- net /LED_CAN_TX: track 15.5 -> 24.5 mm, vias 0 -> 2
- net /MTR_ENABLE: track 113.0 -> 118.8 mm
- net +12V: track 341.1 -> 346.4 mm
- net +3V3: track 484.1 -> 479.3 mm
- net +12VA: track 53.8 -> 58.2 mm
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Other:
- board text added: "Ignición"
- board text added: "REV 2"
- board text added: "®"
- board text removed: "Ignicion"
- board text removed: "REV 1"

Commit message: update vr inputs
Parts:
- added Q4: SS8050, Package_TO_SOT_SMD:SOT-23, F.Cu at (60.8, 96.6)
- added Q7: AO3400A, Package_TO_SOT_SMD:SOT-23, F.Cu at (57.3, 96.6)
- added R68: 1k, Resistor_SMD:R_0603_1608Metric, F.Cu at (56.8, 93.7)
- added R69: 100k, Resistor_SMD:R_0603_1608Metric, F.Cu at (59.9, 93.7)
- C8: value 4700pF -> 4.7nF
- R16, R55, R56, R57, R58: footprint Resistor_SMD:R_0805_2012Metric -> Resistor_SMD:R_0603_1608Metric
- moved R56 6.15 mm to (98.5, 131.9), turned to 90 degrees
- moved R55 5.86 mm to (104.4, 131.9), turned to -90 degrees
- turned R57 to -90 degrees
Connections:
- net PROTO-5 renamed CEL-OUT
- R55 pad 1: /idle -> GND
- R55 pad 2: GND -> /boost
- R56 pad 1: GND -> /idle
- R56 pad 2: /boost -> GND
- R57 pad 1: Net-(U18-IN1) -> /idle
- R57 pad 2: /idle -> Net-(U18-IN1)
- U13 pad 15: unconnected-(U13-PC0-Pad15) -> /CEL_OUT
Routing:
- net /CEL_OUT: track 0.00 -> 103.2 mm, vias 0 -> 3
- net Net-(Q4-B): track 0.00 -> 9.71 mm, vias 0 -> 2
- net Net-(Q4-C): track 0.00 -> 7.20 mm
- net CEL-OUT: track 40.0 -> 46.9 mm
- net +12V: track 346.4 -> 352.7 mm, vias 7 -> 8
- net GND: track 47.3 -> 45.4 mm
- net Net-(J6-Pin_1): track 65.9 -> 64.1 mm
- net /boost: track 76.6 -> 77.2 mm

Commit message: update footprints
Parts:
- added C10: 100uF ±20% 35V, Capacitor_SMD:CP_Elec_6.3x7.7, F.Cu at (157.5, 137.4)
- added G***: LOGO, LOGO, F.Cu at (134.5, 123.9)
- added G***: LOGO, LOGO, B.Cu at (140.3, 136.7)
- C44, C45: footprint Capacitor_SMD:C_0402_1005Metric -> Capacitor_SMD:C_0805_2012Metric
- moved Churrosoft 5.91 mm to (121.7, 135.6)
- moved C45 2.62 mm to (145.4, 63.2)
- moved C46 0.83 mm to (144.9, 67.7)
- moved TP13 0.78 mm to (143.4, 67.1)
- moved U16 0.78 mm to (142.5, 66.5)
- moved C34 0.77 mm to (146.6, 66.9)
- moved J11 0.77 mm to (89.2, 115.9)
- moved C44 0.66 mm to (139.7, 66.7)
- moved C32 0.17 mm to (137.6, 66.1)
Routing:
- net +12V: track 352.7 -> 366.2 mm
- net GND: track 45.4 -> 55.4 mm
- net VDDA: track 18.7 -> 20.7 mm
- net +5V: track 248.7 -> 249.8 mm
Other:
- board text added: "Diseñado en Argentina"
