File: hw_v1/hw_v1.kicad_pcb (KiCad board)
At the start: 4 copper layers, 116.5 x 98 mm, 248 parts, among them J10 Conn_01x01, J11 Conn_01x01, J12 Delphi_Sicma_24, J13 Delphi_Sicma_24, J14 Conn_01x04, J15 Conn_01x03, J16 47352-1001, J2 Conn_01x05, J3 Conn_01x05, J4 Conn_01x05, J5 Conn_01x03, J6 Conn_01x04, J8 USB_B, J9 Tag connect, Q1 AO3400A, Q2 AO3400A, Q3 FDS6890A, Q4 SS8050, Q5 SS8050, Q6 AO3400A, Q7 AO3400A, SW2 SW_Push, U1 MCZ33810EK, U10 BMP280, U11 L78M05ABDT-TR, U12 LM74800, U13 STM32F407VGTx, U14 TJA1051T-3, U15 25Q16, U16 REF3033, U17 SRV05-4, U18 VNLD5090, U19 L78M05ABDT-TR, U2 TC4424A, U21 ADXL343, U3 TC4424A, U4 MAX9926UAEE+, U5 TPL7407LAPWR, U6 LMV324, U7 LMV324, U8 AMS1117-3.3, U9 SP720ABTG, Y1 32.768kHz, Y2 25MHz

Commit message: wip inventree updates
Parts:
- D11, D3, D6, D8: value D -> 1N4148; footprint Diode_SMD:D_SOD-323_HandSoldering -> Diode_SMD:D_SOD-523
- R1: footprint Resistor_SMD:R_0805_2012Metric -> Resistor_SMD:R_0603_1608Metric
- R18, R19, R20, R28, R29, R30: footprint Resistor_SMD:R_0603_1608Metric -> Resistor_SMD:R_0805_2012Metric
- R2, R3, R4, R5: value 10K 1/2W -> 10k; footprint Resistor_SMD:R_0805_2012Metric -> Resistor_SMD:R_0603_1608Metric
- R62: value 90k -> 48.7k
- R63: value 900R -> 42.2k
- moved D11 1.19 mm to (60.0, 109.4)
- moved D8 0.69 mm to (61.6, 109.4)
- moved D3 0.67 mm to (64.7, 109.4)
- moved D6 0.38 mm to (63.1, 109.4)
- moved C17 0.32 mm to (83.3, 73.8)
- moved R25 0.29 mm to (81.5, 81.6)
- moved R20 0.26 mm to (91.5, 70.9)
- moved C27 0.23 mm to (83.2, 81.6)
- moved R15 0.18 mm to (90.6, 73.4)
- moved C16 0.15 mm to (101.3, 73.5)
- moved R35 0.15 mm to (94.2, 81.6)
- moved R14 0.15 mm to (99.5, 73.5)
- moved R18 0.15 mm to (100.4, 71.0)
- moved C24 0.14 mm to (101.2, 81.5)
- moved R30 0.10 mm to (92.2, 81.6)
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Routing:
- net Net-(U1-GD2): track 16.7 -> 25.8 mm, vias 0 -> 2
- net GND: track 55.4 -> 58.1 mm, vias 31 -> 32
- net Net-(D2-K): track 20.9 -> 22.4 mm
- net Net-(D10-K): track 21.3 -> 20.2 mm
- net /Sensors/CH_MAP_m: track 34.7 -> 35.7 mm
- net /Sensors/CH_TPS_m: track 24.4 -> 25.3 mm
- net Net-(D5-K): track 21.9 -> 22.6 mm
- net INJ-3-OUT: track 40.1 -> 39.6 mm

Commit message: update from inventree
Parts:
- C46: footprint Capacitor_SMD:C_0402_1005Metric -> Capacitor_SMD:C_0805_2012Metric
- D11, D16, D17, D18, D3, D6, D8: value 1N4148 -> 1N5819WS; footprint Diode_SMD:D_SOD-523 -> Diode_SMD:D_SOD-323_HandSoldering
- D29, D30: value D -> S110FA
- moved C34 3.16 mm to (147.3, 63.8)
- moved D11 1.23 mm to (58.8, 109.2)
- moved R12 0.82 mm to (109.1, 78.0)
- moved D8 0.70 mm to (60.9, 109.2)
- moved C46 0.68 mm to (145.5, 68.0)
- moved C45 0.62 mm to (145.2, 63.8)
- moved D17 0.57 mm to (108.6, 73.4)
- moved D16 0.41 mm to (108.6, 81.0)
- moved D3 0.31 mm to (64.9, 109.2)
- moved D18 0.30 mm to (154.2, 67.2)
- moved D6 0.28 mm to (62.9, 109.2)
- moved R13 0.20 mm to (109.3, 70.3)
- moved BT1 0.11 mm to (150.5, 67.9)
- moved R65 0.05 mm to (101.4, 56.3)
Routing:
- net GND: track 58.1 -> 63.3 mm
- net ext_a0_in: track 41.8 -> 44.9 mm
- net Net-(D10-K): track 20.2 -> 22.3 mm
- net Net-(D7-K): track 20.8 -> 22.8 mm
- net ext_a1_in: track 46.8 -> 48.2 mm
- net +5C: track 174.8 -> 173.7 mm
- net Net-(J6-Pin_2): track 63.8 -> 64.5 mm
- net INJ-2-OUT: track 58.2 -> 57.6 mm
- net +3V3: track 479.4 -> 480.0 mm
