File: hw_v1/hw_v1.kicad_sch (KiCad schematic)
At the start: 56 parts, among them J7 104031-0811, J8 USB_B, J9 Tag connect, SW2 SW_Push, U13 STM32F407VGTx, U14 TJA1051T-3, U15 25LCxxx, U16 REF3033, U17 SRV05-4, Y1 32.768kHz, Y2 25MHz

Commit message: finish pcb layout
Connections:
- net SD_CLK: now also RN3.2 (R2.1); no longer RN3.4 (R4.1)
- net SD_DAT1: now also RN3.4 (R4.1); no longer RN3.2 (R2.1)
- net VBATT: no longer BT1.1 (+), D18.1 (K), U13.6 (VBAT)
- net MCU-D0: now reaches U13.35 (PB0)
- net MCU-D1: now reaches U13.36 (PB1)
- new net: BT1.1 (+), D18.1 (K), U13.6 (VBAT)
- no-connect marks 11 -> 9
Other:
- note removed: "PROTO 0/1"
Changed lines of the file:
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@@
 	)
 	(no_connect
-		(at 83.82 93.98)
-	)
-	(no_connect
 		(at 83.82 101.6)
 	)
@@
 	)
 	(no_connect
-		(at 83.82 91.44)
-	)
-	(no_connect
 		(at 83.82 134.62)
 	)
@@
 	)
 	(bus_entry
-		(at 95.25 111.76)
-		(size 2.54 -2.54)
-		(stroke
-			(width 0)
-			(type default)
-		)
-	)
-	(bus_entry
 		(at 199.39 116.84)
 		(size 2.54 -2.54)
@@
 	)
 	(bus_entry
-		(at 238.76 96.52)
-		(size 2.54 2.54)
-		(stroke
-			(width 0)
-			(type default)
-		)
-	)
-	(bus_entry
 		(at 241.3 121.92)
 		(size 2.54 2.54)
@@
 	)
 	(bus_entry
-		(at 238.76 93.98)
-		(size 2.54 2.54)
-		(stroke
-			(width 0)
-			(type default)
-		)
-	)
-	(bus_entry
 		(at 276.86 144.78)
 		(size 2.54 -2.54)
@@
 	)
 	(bus_entry
-		(at 95.25 147.32)
-		(size 2.54 -2.54)
-		(stroke
-			(width 0)
-			(type default)
-		)
-	)
-	(bus_entry
 		(at 278.13 96.52)
 		(size 2.54 -2.54)
@@
 		)
 	)
-	(polyline
-		(pts
-			(xy 82.55 90.17) (xy 92.71 90.17)
-		)
-		(stroke
-			(width 0)
-			(type default)
-		)
-	)
 	(wire
 		(pts
@@
 		)
 	)
-	(polyline
-		(pts
-			(xy 83.82 95.25) (xy 92.71 95.25)
-		)
-		(stroke
-			(width 0)
-			(type default)
-		)
-	)
 	(wire
 		(pts
@@
 	(bus
 		(pts
-			(xy 97.79 121.92) (xy 97.79 144.78)
-		)
-		(stroke
-			(width 0)
-			(type default)
-			(color 194 0 194 1)
-		)
-	)
-	(bus
-		(pts
 			(xy 27.94 170.18) (xy 27.94 187.96)
 		)
@@
 		)
 	)
-	(bus
-		(pts
-			(xy 241.3 99.06) (xy 241.3 121.92)
-		)
-		(stroke
-			(width 0)
-			(type default)
-			(color 194 0 194 1)
-		)
-	)
 	(wire
 		(pts
@@
 	(wire
 		(pts
-			(xy 233.68 96.52) (xy 238.76 96.52)
-		)
-		(stroke
-			(width 0)
-			(type default)
-		)
-	)
-	(wire
-		(pts
 			(xy 248.92 97.79) (xy 248.92 96.52)
 		)
@@
 	(bus
 		(pts
-			(xy 238.76 93.98) (xy 238.76 67.31)
+			(xy 238.76 67.31) (xy 238.76 104.14)
 		)
 		(stroke
@@
 	(bus
 		(pts
-			(xy 97.79 144.78) (xy 97.79 147.32)
+			(xy 97.79 121.92) (xy 97.79 147.32)
 		)
 		(stroke
@@
 		)
 	)
-	(bus
-		(pts
-			(xy 97.79 109.22) (xy 97.79 116.84)
-		)
-		(stroke
-			(width 0)
-			(type default)
-			(color 194 0 194 1)
-		)
-	)
 	(wire
 		(pts
@@
 		)
 	)
-	(bus
-		(pts
-			(xy 241.3 96.52) (xy 241.3 99.06)
-		)
-		(stroke
-			(width 0)
-			(type default)
-			(color 194 0 194 1)
-		)
-	)
 	(wire
 		(pts
@@
 	(bus
 		(pts
-			(xy 238.76 96.52) (xy 238.76 104.14)
-		)
-		(stroke
-			(width 0)
-			(type default)
-			(color 204 102 0 1)
-		)
-	)
-	(bus
-		(pts
 			(xy 201.93 111.76) (xy 201.93 114.3)
 		)
@@
 	(bus
 		(pts
-			(xy 97.79 66.04) (xy 97.79 109.22)
+			(xy 97.79 66.04) (xy 97.79 116.84)
 		)
 		(stroke
@@
 	(bus
 		(pts
-			(xy 238.76 96.52) (xy 238.76 93.98)
-		)
-		(stroke
-			(width 0)
-			(type default)
-			(color 204 102 0 1)
-		)
-	)
-	(bus
-		(pts
 			(xy 279.4 149.86) (xy 279.4 151.13)
 		)
@@
 	(wire
 		(pts
-			(xy 233.68 93.98) (xy 238.76 93.98)
-		)
-		(stroke
-			(width 0)
-			(type default)
-		)
-	)
-	(wire
-		(pts
 			(xy 30.48 154.94) (xy 35.56 154.94)
 		)
@@
 	(bus
 		(pts
-			(xy 241.3 93.98) (xy 241.3 96.52)
+			(xy 241.3 93.98) (xy 241.3 121.92)
 		)
 		(stroke
@@
 		)
 	)
-	(text "PROTO 0/1"
-		(exclude_from_sim no)
-		(at 85.09 93.218 0)
-		(effects
-			(font
-				(size 1.27 1.27)
-			)
-			(justify left)
-		)
-	)
 	(text "VDD"
 		(exclude_from_sim no)
@@
 		)
 	)
-	(label "ACCL_CS"
-		(at 238.76 93.98 180)
-		(fields_autoplaced yes)
-		(effects
-			(font
-				(size 0.8 0.8)
-			)
-			(justify right bottom)
-		)
-	)
 	(label "ECN4"
 		(at 30.48 172.72 0)
@@
 	)
 	(label "SD_DAT1"
-		(at 198.12 39.37 270)
+		(at 203.2 39.37 270)
 		(fields_autoplaced yes)
 		(effects
@@
 		)
 	)
-	(label "BARO_CS"
-		(at 238.76 96.52 180)
-		(fields_autoplaced yes)
-		(effects
-			(font
-				(size 0.8 0.8)
-			)
-			(justify right bottom)
-		)
-	)
 	(label "CKP"
 		(at 243.84 124.46 0)
@@
 		)
 	)
-	(label "ACCL_CS"
-		(at 83.82 111.76 0)
-		(fields_autoplaced yes)
-		(effects
-			(font
-				(size 0.8 0.8)
-			)
-			(justify left bottom)
-		)
-	)
 	(label "MAP"
 		(at 204.47 100.33 180)
@@
 		)
 	)
-	(label "BARO_CS"
-		(at 83.82 147.32 0)
-		(fields_autoplaced yes)
-		(effects
-			(font
-				(size 0.8 0.8)
-			)
-			(justify left bottom)
-		)
-	)
 	(label "SYS_SWCLK"
 		(at 83.82 83.82 0)
@@
 	)
 	(label "SD_CLK"
-		(at 203.2 39.37 270)
+		(at 198.12 39.37 270)
 		(fields_autoplaced yes)
 		(effects
@@
 		)
 	)
+	(global_label "MCU-D0"
+		(shape input)
+		(at 83.82 91.44 0)
+		(effects
+			(font
+				(size 1.27 1.27)
+			)
+			(justify left)
+		)
+		(property "Intersheetrefs" "${INTERSHEET_REFS}"
+			(at 83.82 91.44 0)
+			(effects
+				(font
+					(size 1.27 1.27)
+				)
+				(hide yes)
+			)
+		)
+	)
+	(global_label "BARO_CS"
+		(shape input)
+		(at 95.25 147.32 180)
+		(fields_autoplaced yes)
+		(effects
+			(font
+				(size 0.8 0.8)
+			)
+			(justify right)
+		)
+		(property "Intersheetrefs" "${INTERSHEET_REFS}"
+			(at 88.0745 147.32 0)
+			(effects
+				(font
+					(size 1.27 1.27)
+				)
+				(justify right)
+				(hide yes)
+			)
+		)
+	)
 	(global_label "VBUS"
 		(shape input)
@@
 		)
 	)
+	(global_label "ACCL_CS"
+		(shape input)
+		(at 95.25 111.76 180)
+		(fields_autoplaced yes)
+		(effects
+			(font
+				(size 1.27 1.27)
+			)
+			(justify right)
+		)
+		(property "Intersheetrefs" "${INTERSHEET_REFS}"
+			(at 84.161 111.76 0)
+			(effects
+				(font
+					(size 1.27 1.27)
+				)
+				(justify right)
+				(hide yes)
+			)
+		)
+	)
 	(global_label "USART_2_TX"
 		(shape input)
@@
 		)
 	)
+	(global_label "MCU-D1"
+		(shape input)
+		(at 83.82 93.98 0)
+		(effects
+			(font
+				(size 1.27 1.27)
+			)
+			(justify left)
+		)
+		(property "Intersheetrefs" "${INTERSHEET_REFS}"
+			(at 83.82 93.98 0)
+			(effects
+				(font
+					(size 1.27 1.27)
+				)
+				(hide yes)
+			)
+		)
+	)
 	(global_label "OSC_OUT"
 		(shape input)
@@
 				(hide yes)
 			)
-		)
-	)
-	(global_label "VBATT"
-		(shape input)
-		(at 41.91 29.21 180)
-		(fields_autoplaced yes)
-		(effects
-			(font
-				(size 0.889 0.889)
-			)
-			(justify right)
-		)
-		(property "Intersheetrefs" "${INTERSHEET_REFS}"
-			(at 35.9864 29.21 0)
-			(effects
-				(font
-					(size 1.27 1.27)
-				)
-				(justify right)
-				(hide yes)
-			)

Commit message: update SD card holder to Molex 47352
Parts:
- removed J7: 104031-0811, Connector_Card:microSD_HC_Molex_104031-0811, symbol Library:104031-0811
- removed RN4: 47k, Resistor_SMD:R_Array_Convex_4x0603, symbol Device:R_Pack04
- added J16: 47352-1001, uEFI_v5:MOLEX_47352-1001, symbol uEFI_v5:47352-1001
- J9, JP5, SW2, TP12, TP13, TP7, TP8: now left out of the parts list
- U15: value 25LCxxx -> 25Q16; LCSC C188247 -> (none)
Connections:
- net SD_DAT2 is gone; now on net SPI3_SCk: U13.78 (PC10)
- net +3V3: now also J16.4 (VDD)
- net GND: now also J16.6 (VSS), J16.S1 (SHIELD), J16.S2 (SHIELD), J16.S3 (SHIELD), J16.S4 (SHIELD)
- net fan1: now also U13.97 (PE0); no longer U13.98 (PE1)
- net fuel_pump: now also U13.98 (PE1); no longer U13.97 (PE0)
- net SD_CARD_DETECT: now reaches RN3.1 (R1.1)
- net SD_CARD_DETECT: now also U13.66 (PC9), J16.SW
- net SD_CLK renamed SPI3_MOSI
- net SPI3_MOSI: now also J16.3 (CMD)
- net SD_DAT0 renamed SD_CS
- net SD_CS: now also J16.2 (CD/DATA3); no longer RN3.3 (R3.1)
- net SD_DAT1 renamed SPI3_SCk
- net SPI3_SCk: now also J16.5 (CLK); no longer U13.66 (PC9)
- net SD_DAT3 renamed SPI3_MISO
- net SPI3_MISO: now also RN3.3 (R3.1), J16.7 (DATA0)
- no-connect marks 9 -> 11
Other:
- note added: "CAMBIAR: SPI2 por SPI1 para SD 25q64 por 25q16 SDIO por SPI3"

Commit message: update vr inputs
Connections:
- net CEL_OUT: now reaches U13.15 (PC0)
- no-connect marks 11 -> 10
Other:
- sheet Relay & Power Outputs ports: added CEL_OUT; removed none
- note removed: "CAMBIAR: SPI2 por SPI1 para SD 25q64 por 25q16 SDIO por SPI3"
- note removed: "PC8 ---> DAT0 PC9 ---> DAT1 PC10 --> DAT2 PC11 --> DAT3 PC12 --> CLK PD2 ---> CMD PB6 ---> CD (Card Detection)"
Changed lines of the file:
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@@
 	)
 	(no_connect
-		(at 83.82 134.62)
-	)
-	(no_connect
 		(at 33.02 106.68)
 	)
@@
 	(wire
 		(pts
+			(xy 81.28 134.62) (xy 83.82 134.62)
+		)
+		(stroke
+			(width 0)
+			(type default)
+		)
+	)
+	(wire
+		(pts
 			(xy 81.28 114.3) (xy 83.82 114.3)
 		)
@@
 	(wire
 		(pts
-			(xy 81.28 134.62) (xy 83.82 134.62)
-		)
-		(stroke
-			(width 0)
-			(type default)
-		)
-	)
-	(wire
-		(pts
 			(xy 63.5 38.1) (xy 63.5 40.64)
 		)
@@
 		)
 	)
-	(text "CAMBIAR:\n\nSPI2 por SPI1 para SD\n25q64 por 25q16\n\nSDIO por SPI3"
-		(exclude_from_sim no)
-		(at 297.434 39.624 0)
-		(effects
-			(font
-				(size 3 3)
-			)
-			(justify left)
-		)
-	)
 	(text "MCU VREF"
 		(exclude_from_sim no)
@@
 		)
 	)
-	(text "PC8 ---> DAT0\nPC9 ---> DAT1\nPC10 --> DAT2\nPC11 --> DAT3\nPC12 --> CLK\nPD2 ---> CMD\nPB6 ---> CD (Card Detection)"
-		(exclude_from_sim no)
-		(at 292.862 84.328 0)
-		(effects
-			(font
-				(size 1.27 1.27)
-			)
-			(justify left bottom)
-		)
-	)
 	(text "CAN"
 		(exclude_from_sim no)
@@
 		)
 	)
+	(label "CEL_OUT"
+		(at 233.68 137.16 0)
+		(fields_autoplaced yes)
+		(effects
+			(font
+				(size 1.27 1.27)
+			)
+			(justify left bottom)
+		)
+	)
 	(label "SW_Clutch_m"
 		(at 229.87 156.21 0)
@@
 		)
 	)
+	(label "CEL_OUT"
+		(at 83.82 134.62 0)
+		(fields_autoplaced yes)
+		(effects
+			(font
+				(size 0.8 0.8)
+			)
+			(justify left bottom)
+		)
+	)
 	(label "SPI2_MISO"
 		(at 278.13 96.52 180)
@@
 			(effects
 				(font
+					(size 1.27 1.27)
+				)
+				(justify right)
+			)
+		)
+		(pin "CEL_OUT" input
+			(at 233.68 137.16 0)
+			(effects
+				(font

Commit message: update footprints
Parts:
- C44, C45: footprint Capacitor_SMD:C_0402_1005Metric -> Capacitor_SMD:C_0805_2012Metric
Changed lines of the file:
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@@
 			)
 		)
-		(property "Footprint" "Capacitor_SMD:C_0402_1005Metric"
+		(property "Footprint" "Capacitor_SMD:C_0805_2012Metric"
 			(at 138.1252 189.865 0)
 			(effects
@@
 			)
 		)
-		(property "Footprint" "Capacitor_SMD:C_0402_1005Metric"
+		(property "Footprint" "Capacitor_SMD:C_0805_2012Metric"
 			(at 113.9952 187.325 0)
 			(effects

Commit message: update footprints
Parts:
- D18: LCSC C511874 -> C5277952
Changed lines of the file:
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@@
 			)
 		)
-		(property "LCSC" "C511874"
+		(property "LCSC" "C5277952"
 			(at 38.1 24.13 0)
 			(effects
