File: hw_v1/hw_v1.kicad_sch (KiCad schematic)
At the start: 55 parts, among them J16 47352-1001, J8 USB_B, J9 Tag connect, SW2 SW_Push, U13 STM32F407VGTx, U14 TJA1051T-3, U15 25Q16, U16 REF3033, U17 SRV05-4, Y1 32.768kHz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

Commit message: update from inventree
Parts:
- BT1: LCSC (none) -> C722633; STOCK (none) -> CON-000415-00
- C26, C29: STOCK (none) -> CAP-000176-00
- C30, C31, C32, C33, C35, C36, C37, C39: STOCK (none) -> CAP-000175-00
- C34: STOCK (none) -> CAP-000328-00
- C38: STOCK (none) -> CAP-000055-00
- C40, C41: STOCK (none) -> CAP-000329-00
- C42, C43: STOCK (none) -> CAP-000123-00
- C44, C45: STOCK (none) -> CAP-000100-00
- C46: footprint Capacitor_SMD:C_0402_1005Metric -> Capacitor_SMD:C_0805_2012Metric; LCSC C1525 -> C38141; STOCK (none) -> CAP-000325-00
- D18: value 1N4148 -> 1N5819WS; footprint Diode_SMD:D_SOD-523 -> Diode_SMD:D_SOD-323_HandSoldering; LCSC C5277952 -> C191023; STOCK (none) -> DIO-000272-00
- D19: STOCK (none) -> DIO-000272-00
- J16: LCSC (none) -> C293569; STOCK (none) -> CON-000335-00
- J8: STOCK (none) -> CON-000152-00
- J9, JP5, TP12, TP13, TP7, TP8: now not fitted
- R27: LCSC C25804 -> C115324; STOCK (none) -> RES-000118-00
- R31: STOCK (none) -> RES-000343-00
- R32, R34, R37, R38, R42, R43, R44: STOCK (none) -> RES-000117-00
- RN3: STOCK (none) -> RES-000354-00
- SW2: LCSC (none) -> C412370; STOCK (none) -> MEC-000125-00
- U13: STOCK (none) -> ICS-000003-00
- U14: STOCK (none) -> ICS-000359-00
- U15: LCSC (none) -> C82317; STOCK (none) -> ICS-000015-00
- U16: STOCK (none) -> PWR-000360-00
- U17: STOCK (none) -> DIO-000361-00
- Y1: STOCK (none) -> CLK-000364-00
- Y2: STOCK (none) -> CLK-000106-00
