File: hw_v1/relays.kicad_sch (KiCad schematic)
At the start: 19 parts, among them J10 Conn_01x01, J11 Conn_01x01, Q5 SS8050, Q6 AO3400A, U18 VNLD5090, U5 TPL7407LAPWR

Commit message: wip pcb layout
Other:
- note added: "El pin de Fault se utiliza para el homming: al setear una corriente baja, al chocar contra el multiple de admision tendria que subir la corriente del motor => probancando una falla en el driver"
- note added: "TODO: estaria bueno agregarle un led a estas salidas"
Changed lines of the file:
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@@
+		)
+	)
+	(text "El pin de Fault se utiliza para el homming:\nal setear una corriente baja, al chocar contra el multiple de admision\ntendria que subir la corriente del motor => probancando una falla en el driver"
+		(exclude_from_sim no)
+		(at 64.008 193.04 0)
+		(effects
+			(font
+				(size 1.27 1.27)
+			)
+			(justify left)
+		)
+	)
+	(text "TODO:\nestaria bueno agregarle un led a estas salidas"
+		(exclude_from_sim no)
+		(at 65.278 51.562 0)
+		(effects
+			(font
+				(size 4 4)
+			)
+			(justify left)
 		)
 	)

Commit message: finish pcb layout
Connections:
- net 12V-SW is gone; now on net +12V: D29.1 (K), D30.1 (K)
- net STEP-A1 renamed STEPPER-A1
- net STEP-A2 renamed STEPPER-A2
- net STEP-B1 renamed STEPPER-B1
- net STEP-B2 renamed STEPPER-B2
Changed lines of the file:
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@@
 	(wire
 		(pts
-			(xy 248.92 152.4) (xy 254 152.4)
+			(xy 248.92 152.4) (xy 257.81 152.4)
 		)
 		(stroke
@@
 			)
 			(justify left bottom)
-		)
-	)
-	(global_label "12V-SW"
-		(shape input)
-		(at 254 118.11 0)
-		(effects
-			(font
-				(size 1.27 1.27)
-			)
-			(justify left)
-		)
-		(property "Intersheetrefs" "${INTERSHEET_REFS}"
-			(at 254 118.11 0)
-			(effects
-				(font
-					(size 1.27 1.27)
-				)
-				(hide yes)
-			)
 		)
 	)
@@
 		)
 	)
+	(global_label "STEPPER-B1"
+		(shape input)
+		(at 109.22 166.37 0)
+		(fields_autoplaced yes)
+		(effects
+			(font
+				(size 1.27 1.27)
+			)
+			(justify left)
+		)
+		(property "Intersheetrefs" "${INTERSHEET_REFS}"
+			(at 124.5422 166.37 0)
+			(effects
+				(font
+					(size 1.27 1.27)
+				)
+				(justify left)
+				(hide yes)
+			)
+		)
+	)
 	(global_label "FUELPUMP-OUT"
 		(shape input)
@@
 		)
 	)
-	(global_label "STEP-A2"
+	(global_label "STEPPER-A1"
 		(shape input)
-		(at 109.22 161.29 0)
+		(at 109.22 158.75 0)
+		(fields_autoplaced yes)
 		(effects
 			(font
@@
 		)
 		(property "Intersheetrefs" "${INTERSHEET_REFS}"
-			(at 109.22 161.29 0)
-			(effects
-				(font
-					(size 1.27 1.27)
-				)
-				(hide yes)
-			)
-		)
-	)
-	(global_label "STEP-B1"
+			(at 124.3608 158.75 0)
+			(effects
+				(font
+					(size 1.27 1.27)
+				)
+				(justify left)
+				(hide yes)
+			)
+		)
+	)
+	(global_label "STEPPER-B2"
 		(shape input)
-		(at 109.22 166.37 0)
+		(at 109.22 168.91 0)
+		(fields_autoplaced yes)
 		(effects
 			(font
@@
 		)
 		(property "Intersheetrefs" "${INTERSHEET_REFS}"
-			(at 109.22 166.37 0)
-			(effects
-				(font
-					(size 1.27 1.27)
-				)
-				(hide yes)
-			)
-		)
-	)
-	(global_label "STEP-B2"
+			(at 124.5422 168.91 0)
+			(effects
+				(font
+					(size 1.27 1.27)
+				)
+				(justify left)
+				(hide yes)
+			)
+		)
+	)
+	(global_label "STEPPER-A2"
 		(shape input)
-		(at 109.22 168.91 0)
+		(at 109.22 161.29 0)
+		(fields_autoplaced yes)
 		(effects
 			(font
@@
 		)
 		(property "Intersheetrefs" "${INTERSHEET_REFS}"
-			(at 109.22 168.91 0)
-			(effects
-				(font
-					(size 1.27 1.27)
-				)
-				(hide yes)
-			)
-		)
-	)
-	(global_label "12V-SW"
-		(shape input)
-		(at 254 152.4 0)
-		(effects
-			(font
-				(size 1.27 1.27)
-			)
-			(justify left)
-		)
-		(property "Intersheetrefs" "${INTERSHEET_REFS}"
-			(at 254 152.4 0)
-			(effects
-				(font
-					(size 1.27 1.27)
-				)
+			(at 124.3608 161.29 0)
+			(effects
+				(font
+					(size 1.27 1.27)
+				)
+				(justify left)
 				(hide yes)
 			)
@@
 		(property "Intersheetrefs" "${INTERSHEET_REFS}"
 			(at 185.42 76.2 0)
-			(effects
-				(font
-					(size 1.27 1.27)
-				)
-				(hide yes)
-			)
-		)
-	)
-	(global_label "STEP-A1"
-		(shape input)
-		(at 109.22 158.75 0)
-		(effects
-			(font
-				(size 1.27 1.27)
-			)
-			(justify left)
-		)
-		(property "Intersheetrefs" "${INTERSHEET_REFS}"
-			(at 109.22 158.75 0)
 			(effects
 				(font
@@
 	)
 	(symbol
+		(lib_id "power:+12V")
+		(at 257.81 152.4 0)
+		(unit 1)
+		(exclude_from_sim no)
+		(in_bom yes)
+		(on_board yes)
+		(dnp no)
+		(fields_autoplaced yes)
+		(property "Reference" "#PWR0174"
+			(at 257.81 156.21 0)
+			(effects
+				(font
+					(size 1.27 1.27)
+				)
+				(hide yes)
+			)
+		)
+		(property "Value" "+12V"
+			(at 257.81 147.32 0)
+			(effects
+				(font
+					(size 1.27 1.27)
+				)
+			)
+		)
+		(property "Footprint" ""
+			(at 257.81 152.4 0)
+			(effects
+				(font
+					(size 1.27 1.27)
+				)
+				(hide yes)
+			)
+		)
+		(property "Datasheet" ""
+			(at 257.81 152.4 0)
+			(effects
+				(font
+					(size 1.27 1.27)
+				)
+				(hide yes)
+			)
+		)
+		(property "Description" "Power symbol creates a global label with name \"+12V\""
+			(at 257.81 152.4 0)
+			(effects
+				(font
+					(size 1.27 1.27)
+				)
+				(hide yes)
+			)
+		)
+		(pin "1"
+		)
+		(instances
+			(project "hw_v1"
+				(path "/b3feb07e-be80-40e1-bd13-6cd54c2f8b0c/aca74028-30ce-4304-a4a8-c39cedc5a58f"
+					(reference "#PWR0174")
+					(unit 1)
+				)
+			)
+		)
+	)
+	(symbol
 		(lib_id "Device:R")
 		(at 205.74 137.16 270)
@@
 					(unit 1)
 				)
+			)
+		)
+	)
+	(symbol
+		(lib_id "power:+12V")
+		(at 254 118.11 0)
+		(unit 1)
+		(exclude_from_sim no)
+		(in_bom yes)
+		(on_board yes)
+		(dnp no)
+		(fields_autoplaced yes)
+		(property "Reference" "#PWR0173"
+			(at 254 121.92 0)
+			(effects
+				(font
+					(size 1.27 1.27)
+				)
+				(hide yes)
+			)
+		)
+		(property "Value" "+12V"
+			(at 254 113.03 0)
+			(effects
+				(font
+					(size 1.27 1.27)
+				)
+			)
+		)
+		(property "Footprint" ""
+			(at 254 118.11 0)
+			(effects
+				(font
+					(size 1.27 1.27)
+				)
+				(hide yes)
+			)
+		)
+		(property "Datasheet" ""
+			(at 254 118.11 0)
+			(effects
+				(font
+					(size 1.27 1.27)
+				)
+				(hide yes)
+			)
+		)
+		(property "Description" "Power symbol creates a global label with name \"+12V\""
+			(at 254 118.11 0)
+			(effects
+				(font
+					(size 1.27 1.27)
+				)
+				(hide yes)
+			)
+		)
+		(pin "1"
+		)
+		(instances
+			(project "hw_v1"
+				(path "/b3feb07e-be80-40e1-bd13-6cd54c2f8b0c/aca74028-30ce-4304-a4a8-c39cedc5a58f"
+					(reference "#PWR0173")
+					(unit 1)
+				)

Commit message: update SD card holder to Molex 47352
Parts:
- A1, J10, J11, JP6, JP7, JP8: now left out of the parts list
- D29, D30: LCSC (none) -> C556397
Changed lines of the file:
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@@
 	(version 20231120)
 	(generator "eeschema")
-	(generator_version "7.99")
+	(generator_version "8.0")
 	(paper "A4")
 	(title_block
 		(title "μEFI (Speeduino FW compatible)")
 		(date "2023-12-25")
-		(rev "v6")
+		(rev "v6.1")
 		(company "Churrosoft ®")
-		(comment 1 "CERN-OHL-S-2.0 license\n")
+		(comment 1 "CERN-OHL-S-2.0 license")
 	)
 	(junction
@@
 		(unit 1)
 		(exclude_from_sim no)
-		(in_bom yes)
+		(in_bom no)
 		(on_board yes)
 		(dnp no)
@@
 		(unit 1)
 		(exclude_from_sim no)
-		(in_bom yes)
+		(in_bom no)
 		(on_board yes)
 		(dnp no)
@@
 		(unit 1)
 		(exclude_from_sim no)
-		(in_bom yes)
+		(in_bom no)
 		(on_board yes)
 		(dnp no)
@@
 		(unit 1)
 		(exclude_from_sim no)
-		(in_bom yes)
+		(in_bom no)
 		(on_board yes)
 		(dnp no)
@@
 			)
 		)
+		(property "LCSC" "C556397"
+			(at 248.92 146.05 90)
+			(effects
+				(font
+					(size 1.27 1.27)
+				)
+				(hide yes)
+			)
+		)
+		(property "Field10" ""
+			(at 248.92 146.05 90)
+			(effects
+				(font
+					(size 1.27 1.27)
+				)
+				(hide yes)
+			)
+		)
 		(pin "1"
 		)
@@
 		(unit 1)
 		(exclude_from_sim no)
-		(in_bom yes)
+		(in_bom no)
 		(on_board yes)
 		(dnp no)
@@
 		(unit 1)
 		(exclude_from_sim no)
-		(in_bom yes)
+		(in_bom no)
 		(on_board yes)
 		(dnp no)
@@
 			(effects
 				(font
+					(size 1.27 1.27)
+				)
+				(hide yes)
+			)
+		)
+		(property "LCSC" "C556397"
+			(at 248.92 124.46 90)
+			(effects
+				(font
+					(size 1.27 1.27)
+				)
+				(hide yes)
+			)
+		)
+		(property "Field10" ""
+			(at 248.92 124.46 90)
+			(effects
+				(font

Commit message: update vr inputs
Parts:
- added Q4: SS8050, Package_TO_SOT_SMD:SOT-23, symbol Transistor_BJT:2N3055
- added Q7: AO3400A, Package_TO_SOT_SMD:SOT-23, symbol Transistor_FET:AO3400A
- added R68: 1k, Resistor_SMD:R_0603_1608Metric, symbol Device:R
- added R69: 100k, Resistor_SMD:R_0603_1608Metric, symbol Device:R
- R55, R56: footprint Resistor_SMD:R_0805_2012Metric -> Resistor_SMD:R_0603_1608Metric; Digikey Part Number 311-100KCRCT-ND -> (none); LCSC (none) -> C25803; Manufacturer_Name Yageo -> (none); Manufacturer_Part_Number RC0805FR-07100KL -> (none); STOCK (none) -> 44; URL https://www.digikey.com/product-detail/en/yageo/RC0805FR-07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 -> (none)
- R57, R58: footprint Resistor_SMD:R_0805_2012Metric -> Resistor_SMD:R_0603_1608Metric; LCSC (none) -> C21190; URL https://www.digikey.com/product-detail/en/yageo/RC0805FR-07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 -> (none)
- U18: LCSC (none) -> C222209
Connections:
- net +12V: now also R69.1
- net GND: now also R55.1, R56.2, Q4.2 (E), Q7.2 (S); no longer R55.2, R56.1
- net boost: now also R55.2; no longer R56.2
- net idle: now also R56.1, R57.1; no longer R55.1, R57.2
- net at U18.1 (IN1): now also R57.2; no longer R57.1
- new net: Q4.3 (C), Q7.1 (G), R69.2
- new net: Q4.1 (B), R68.2
- new net CEL-OUT: Q7.3 (D)
- new net CEL_OUT: R68.1

Commit message: update footprints
Parts:
- added C10: 100uF ±20% 35V, Capacitor_SMD:CP_Elec_6.3x7.7, symbol Device:CP_Small
Connections:
- net +12V: now also C10.1
- net GND: now also C10.2
Changed lines of the file:
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@@
 	(wire
 		(pts
+			(xy 96.52 143.51) (xy 96.52 146.05)
+		)
+		(stroke
+			(width 0)
+			(type default)
+		)
+	)
+	(wire
+		(pts
 			(xy 177.8 76.2) (xy 177.8 77.47)
 		)
@@
 	(symbol
 		(lib_id "power:+12V")
-		(at 96.52 146.05 0)
+		(at 96.52 143.51 0)
 		(unit 1)
 		(exclude_from_sim no)
@@
 		(fields_autoplaced yes)
 		(property "Reference" "#PWR0139"
-			(at 96.52 149.86 0)
+			(at 96.52 147.32 0)
 			(effects
 				(font
@@
 		)
 		(property "Value" "+12V"
-			(at 96.52 140.97 0)
+			(at 96.52 138.43 0)
 			(effects
 				(font
@@
 		)
 		(property "Footprint" ""
-			(at 96.52 146.05 0)
+			(at 96.52 143.51 0)
 			(effects
 				(font
@@
 		)
 		(property "Datasheet" ""
-			(at 96.52 146.05 0)
+			(at 96.52 143.51 0)
 			(effects
 				(font
@@
 		)
 		(property "Description" ""
-			(at 96.52 146.05 0)
+			(at 96.52 143.51 0)
 			(effects
 				(font
@@
 	)
 	(symbol
+		(lib_id "power:+12V")
+		(at 114.3 144.78 0)
+		(unit 1)
+		(exclude_from_sim no)
+		(in_bom yes)
+		(on_board yes)
+		(dnp no)
+		(fields_autoplaced yes)
+		(property "Reference" "#PWR0179"
+			(at 114.3 148.59 0)
+			(effects
+				(font
+					(size 1.27 1.27)
+				)
+				(hide yes)
+			)
+		)
+		(property "Value" "+12V"
+			(at 114.3 139.7 0)
+			(effects
+				(font
+					(size 1.27 1.27)
+				)
+			)
+		)
+		(property "Footprint" ""
+			(at 114.3 144.78 0)
+			(effects
+				(font
+					(size 1.27 1.27)
+				)
+				(hide yes)
+			)
+		)
+		(property "Datasheet" ""
+			(at 114.3 144.78 0)
+			(effects
+				(font
+					(size 1.27 1.27)
+				)
+				(hide yes)
+			)
+		)
+		(property "Description" ""
+			(at 114.3 144.78 0)
+			(effects
+				(font
+					(size 1.27 1.27)
+				)
+				(hide yes)
+			)
+		)
+		(pin "1"
+		)
+		(instances
+			(project "hw_v1"
+				(path "/b3feb07e-be80-40e1-bd13-6cd54c2f8b0c/aca74028-30ce-4304-a4a8-c39cedc5a58f"
+					(reference "#PWR0179")
+					(unit 1)
+				)
+			)
+		)
+	)
+	(symbol
 		(lib_id "Device:R")
 		(at 153.67 88.9 90)
@@
 					(unit 1)
 				)
+			)
+		)
+	)
+	(symbol
+		(lib_id "Device:CP_Small")
+		(at 114.3 147.32 0)
+		(unit 1)
+		(exclude_from_sim no)
+		(in_bom yes)
+		(on_board yes)
+		(dnp no)
+		(property "Reference" "C10"
+			(at 116.5352 146.1516 0)
+			(effects
+				(font
+					(size 1.27 1.27)
+				)
+				(justify left)
+			)
+		)
+		(property "Value" "100uF ±20% 35V"
+			(at 116.5352 148.463 0)
+			(effects
+				(font
+					(size 1.27 1.27)
+				)
+				(justify left)
+			)
+		)
+		(property "Footprint" "Capacitor_SMD:CP_Elec_6.3x7.7"
+			(at 114.3 147.32 0)
+			(effects
+				(font
+					(size 1.27 1.27)
+				)
+				(hide yes)
+			)
+		)
+		(property "Datasheet" "~"
+			(at 114.3 147.32 0)
+			(effects
+				(font
+					(size 1.27 1.27)
+				)
+				(hide yes)
+			)
+		)
+		(property "Description" ""
+			(at 114.3 147.32 0)
+			(effects
+				(font
+					(size 1.27 1.27)
+				)
+				(hide yes)
+			)
+		)
+		(property "LCSC" "C141427"
+			(at 114.3 147.32 0)
+			(effects
+				(font
+					(size 0.889 0.889)
+				)
+				(hide yes)
+			)
+		)
+		(pin "1"
+		)
+		(pin "2"
+		)
+		(instances
+			(project "hw_v1"
+				(path "/b3feb07e-be80-40e1-bd13-6cd54c2f8b0c/aca74028-30ce-4304-a4a8-c39cedc5a58f"
+					(reference "C10")
+					(unit 1)
+				)
+			)
+		)
+	)
+	(symbol
+		(lib_id "power:GND")
+		(at 114.3 149.86 0)
+		(unit 1)
+		(exclude_from_sim no)
+		(in_bom yes)
+		(on_board yes)
+		(dnp no)
+		(property "Reference" "#PWR0180"
+			(at 114.3 156.21 0)
+			(effects
+				(font
+					(size 1.27 1.27)
+				)
+				(hide yes)
+			)
+		)
+		(property "Value" "GND"
+			(at 114.427 154.2542 0)
+			(effects
+				(font
+					(size 1.27 1.27)
+				)
+			)
+		)
+		(property "Footprint" ""
+			(at 114.3 149.86 0)
+			(effects
+				(font
+					(size 1.27 1.27)
+				)
+				(hide yes)
+			)
+		)
+		(property "Datasheet" ""
+			(at 114.3 149.86 0)
+			(effects
+				(font
+					(size 1.27 1.27)
+				)
+				(hide yes)
+			)
+		)
+		(property "Description" ""
+			(at 114.3 149.86 0)
+			(effects
+				(font
+					(size 1.27 1.27)
+				)
+				(hide yes)
+			)
+		)
+		(pin "1"
+		)
+		(instances
+			(project "hw_v1"
+				(path "/b3feb07e-be80-40e1-bd13-6cd54c2f8b0c/aca74028-30ce-4304-a4a8-c39cedc5a58f"
+					(reference "#PWR0180")
+					(unit 1)
+				)

Commit message: update from inventree
Parts:
- A1: LCSC (none) -> -; STOCK (none) -> MOD-000414-00
- C10: STOCK (none) -> CAP-000179-00
- D28: STOCK BI000000597 -> DIO-000157-00
- D29, D30: value D -> S110FA; STOCK (none) -> DIO-000332-00
- J10, J11, JP6, JP7, JP8: now not fitted
- Q4, Q5: STOCK (none) -> TRA-000056-00
- Q6, Q7: STOCK (none) -> TRA-000186-00
- R53, R57, R58, R68: STOCK (none) -> RES-000107-00
- R54, R55, R56, R69: STOCK 44 -> RES-000229-00
- U18: STOCK (none) -> TRA-000362-00
- U5: STOCK (none) -> TRA-000031-00
Changed lines of the file:
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@@
 			)
 		)
+		(property "STOCK" "TRA-000186-00"
+			(at 233.68 87.63 0)
+			(effects
+				(font
+					(size 1.27 1.27)
+				)
+				(hide yes)
+			)
+		)
 		(pin "1"
 		)
@@
 			)
 		)
+		(property "STOCK" "RES-000107-00"
+			(at 205.74 129.54 0)
+			(effects
+				(font
+					(size 1.27 1.27)
+				)
+				(hide yes)
+			)
+		)
 		(pin "1"
 		)
@@
 		(in_bom no)
 		(on_board yes)
-		(dnp no)
+		(dnp yes)
 		(property "Reference" "J10"
 			(at 70.866 86.614 0)
@@
 		(in_bom no)
 		(on_board yes)
-		(dnp no)
+		(dnp yes)
 		(fields_autoplaced yes)
 		(property "Reference" "JP7"
@@
 			)
 		)
-		(property "STOCK" "44"
+		(property "STOCK" "RES-000229-00"
 			(at 196.85 144.78 90)
 			(effects
@@
 			)
 		)
+		(property "STOCK" "TRA-000031-00"
+			(at 97.155 78.105 0)
+			(effects
+				(font
+					(size 1.27 1.27)
+				)
+				(hide yes)
+			)
+		)
 		(pin "1"
 		)
@@
 			)
 		)
+		(property "STOCK" "TRA-000056-00"
+			(at 163.83 88.9 0)
+			(effects
+				(font
+					(size 1.27 1.27)
+				)
+				(hide yes)
+			)
+		)
 		(pin "1"
 		)
@@
 		(in_bom no)
 		(on_board yes)
-		(dnp no)
+		(dnp yes)
 		(fields_autoplaced yes)
 		(property "Reference" "JP8"
@@
 			)
 		)
-		(property "STOCK" "44"
+		(property "STOCK" "RES-000229-00"
 			(at 161.29 76.2 90)
 			(effects
@@
 			)
 		)
+		(property "STOCK" "RES-000107-00"
+			(at 212.09 93.98 0)
+			(effects
+				(font
+					(size 1.27 1.27)
+				)
+				(hide yes)
+			)
+		)
 		(pin "1"
 		)
@@
 			)
 		)
-		(property "STOCK" "BI000000597"
+		(property "STOCK" "DIO-000157-00"
 			(at 182.88 82.55 0)
 			(effects
@@
 			)
 		)
+		(property "STOCK" "RES-000107-00"
+			(at 153.67 88.9 0)
+			(effects
+				(font
+					(size 1.27 1.27)
+				)
+				(hide yes)
+			)
+		)
 		(pin "1"
 		)
@@
 		(in_bom no)
 		(on_board yes)
-		(dnp no)
+		(dnp yes)
 		(fields_autoplaced yes)
 		(property "Reference" "JP6"
@@
 			)
 		)
+		(property "STOCK" "TRA-000186-00"
+			(at 175.26 82.55 0)
+			(effects
+				(font
+					(size 1.27 1.27)
+				)
+				(hide yes)
+			)
+		)
 		(pin "1"
 		)
@@
 			)
 		)
+		(property "STOCK" "CAP-000179-00"
+			(at 114.3 147.32 0)
+			(effects
+				(font
+					(size 1.27 1.27)
+				)
+				(hide yes)
+			)
+		)
 		(pin "1"
 		)
@@
 			)
 		)
-		(property "STOCK" "44"
+		(property "STOCK" "RES-000229-00"
 			(at 219.71 81.28 90)
 			(effects
@@
 			)
 		)
-		(property "Value" "D"
+		(property "Value" "S110FA"
 			(at 250.9266 144.907 90)
 			(effects
@@
 			)
 		)
+		(property "STOCK" "DIO-000332-00"
+			(at 248.92 146.05 0)
+			(effects
+				(font
+					(size 1.27 1.27)
+				)
+				(hide yes)
+			)
+		)
 		(pin "1"
 		)
@@
 		(in_bom no)
 		(on_board yes)
-		(dnp no)
+		(dnp yes)
 		(property "Reference" "J11"
 			(at 119.126 96.012 0)
@@
 			)
 		)
+		(property "LCSC" "-"
+			(at 96.52 161.29 0)
+			(effects
+				(font
+					(size 1.27 1.27)
+				)
+				(hide yes)
+			)
+		)
+		(property "STOCK" "MOD-000414-00"
+			(at 96.52 161.29 0)
+			(effects
+				(font
+					(size 1.27 1.27)
+				)
+				(hide yes)
+			)
+		)
 		(pin "7"
 		)
@@
 			)
 		)
+		(property "STOCK" "TRA-000056-00"
+			(at 222.25 93.98 0)
+			(effects
+				(font
+					(size 1.27 1.27)
+				)
+				(hide yes)
+			)
+		)
 		(pin "1"
 		)
@@
 			)
 		)
-		(property "STOCK" "44"
+		(property "STOCK" "RES-000229-00"
 			(at 196.85 121.92 90)
 			(effects
@@
 			)
 		)
-		(property "Value" "D"
+		(property "Value" "S110FA"
 			(at 250.9266 125.603 90)
 			(effects
@@
 			)
 		)
+		(property "STOCK" "DIO-000332-00"
+			(at 248.92 124.46 0)
+			(effects
+				(font
+					(size 1.27 1.27)
+				)
+				(hide yes)
+			)
+		)
 		(pin "1"
 		)
@@
 			)
 		)
+		(property "STOCK" "RES-000107-00"
+			(at 205.74 137.16 0)
+			(effects
+				(font
+					(size 1.27 1.27)
+				)
+				(hide yes)
+			)
+		)
 		(pin "1"
 		)
@@
 			(at 223.52 134.62 0)
 			(effects
+				(font
+					(size 1.27 1.27)
+				)
+				(hide yes)
+			)
+		)
+		(property "STOCK" "TRA-000362-00"
+			(at 223.52 134.62 0)
+			(effects
