File: hw_v1/sensors.kicad_sch (KiCad schematic)
At the start: 49 parts, among them U10 BMP280, U6 LMV324, U7 LMV324, U9 SP720ABTG

Commit message: wip pcb layout
Parts:
- added C47, C50: 100nF, Capacitor_SMD:C_0805_2012Metric, symbol Device:C_Small
- added U21: ADXL343, Package_LGA:LGA-14_3x5mm_P0.8mm_LayoutBorder1x6y, symbol Sensor_Motion:ADXL343
Connections:
- net +3V3: now also C47.1, C50.1, U21.1 (Vdd_I/O), U21.6 (Vs)
- net GND: now also R23.2, R26.2, C47.2, C50.2, U21.2 (GND), U21.4 (GND), U21.5 (GND)
- net SPI2_MISO: now also U21.12 (SDO/ADDR)
- net SPI2_MOSI: now also U21.13 (SDA/SDI/SDIO)
- net SPI2_SCK: now also U21.14 (SCL/SCLK)
- net ext_a0_in: now also R24.2
- net ext_a0_out: now also U7.13 (-), U7.14
- net ext_a1_in: now also R17.2
- net ext_a1_out: now also U7.8, U7.9 (-)
- net at R24.1: now also R26.1, U7.12 (+)
- net at R23.1: now also R17.1, U7.10 (+)
- net CH_CLT renamed CLT_Sensor
- net CH_IAT renamed IAT_Sensor
- net CH_O2 renamed O2_Sensor
- net CH_TPS renamed TPS_Sensor
- new net ACCL_CS: U21.7 (~{CS})
- no-connect marks 6 -> 0
Other:
- note added: "Accelerometer"
- note added: "Barometer"
- note removed: "TODO: internal map selector map interno / externo (con unos jumpers soldables"
- moved on the sheet: C13, C18, R15, R17, R20, R23, R24, R26, R33, R35, R39, R40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

Commit message: wip sensors traces, added can
Connections:
- net CH_MAP renamed MAP_Sensor
Changed lines of the file:
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@@
+		)
+	)
+	(global_label "ext_a1_in"
+		(shape input)
+		(at 156.21 109.22 180)
+		(fields_autoplaced yes)
+		(effects
+			(font
+				(size 1.27 1.27)
+			)
+			(justify right)
+		)
+		(property "Intersheetrefs" "${INTERSHEET_REFS}"
+			(at 144.3349 109.22 0)
+			(effects
+				(font
+					(size 1.27 1.27)
+				)
+				(justify right)
+				(hide yes)
+			)
 		)
 	)
@@
 		)
 	)
+	(global_label "MAP_Sensor"
+		(shape input)
+		(at 29.21 111.76 180)
+		(effects
+			(font
+				(size 0.8 0.8)
+			)
+			(justify right)
+		)
+		(property "Intersheetrefs" "${INTERSHEET_REFS}"
+			(at 29.21 111.76 0)
+			(effects
+				(font
+					(size 1.27 1.27)
+				)
+				(hide yes)
+			)
+		)
+	)
 	(global_label "IAT_Sensor"
 		(shape input)
@@
 		)
 	)
-	(global_label "CH_MAP"
-		(shape input)
-		(at 28.575 111.76 180)
-		(effects
-			(font
-				(size 0.889 0.889)
-			)
-			(justify right)
-		)
-		(property "Intersheetrefs" "${INTERSHEET_REFS}"
-			(at 25.235 111.7045 0)
-			(effects
-				(font
-					(size 0.889 0.889)
+	(global_label "ext_a0_in"
+		(shape input)
+		(at 113.03 109.22 180)
+		(fields_autoplaced yes)
+		(effects
+			(font
+				(size 1.27 1.27)
+			)
+			(justify right)
+		)
+		(property "Intersheetrefs" "${INTERSHEET_REFS}"
+			(at 101.1549 109.22 0)
+			(effects
+				(font
+					(size 1.27 1.27)
 				)
 				(justify right)
@@
 		)
 	)
-	(hierarchical_label "ext_a0_in"
-		(shape input)
-		(at 113.03 109.22 180)
-		(fields_autoplaced yes)
-		(effects
-			(font
-				(size 1.27 1.27)
-			)
-			(justify right)
-		)
-	)
 	(hierarchical_label "SPI2_MISO"
 		(shape input)
@@
 		(fields_autoplaced yes)
 		(effects
-			(font
-				(size 1.27 1.27)
-			)
-			(justify right)
-		)
-	)
-	(hierarchical_label "ext_a1_in"
-		(shape input)
-		(at 156.21 109.22 180)
-		(fields_autoplaced yes)
-		(effects

Commit message: placed al SMD, wip pmic traces
Connections:
- net AUX_CH6_m is gone; now on net ext_a0_in: U9.12 (I11)
- net AUX_CH8_m is gone; now on net ext_a1_in: U9.13 (I12)
- net AUX_CH1_m: no longer names the net of U9.4 (I4)
- net AUX_CH2_m: no longer names the net of U9.3 (I3)
- net AUX_CH3_m: no longer names the net of U9.2 (I2)
- net AUX_CH4_m: no longer names the net of U9.5 (I5)
- net AUX_CH5_m: no longer names the net of U9.1 (I1)
Changed lines of the file:
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@@
-		)
-	)
-	(label "AUX_CH6_m"
-		(at 245.11 100.33 0)
-		(fields_autoplaced yes)
-		(effects
-			(font
-				(size 0.889 0.889)
-			)
-			(justify left bottom)
-		)
-	)
-	(label "AUX_CH4_m"
-		(at 224.79 102.87 180)
-		(fields_autoplaced yes)
-		(effects
-			(font
-				(size 0.889 0.889)
-			)
-			(justify right bottom)
 		)
 	)
@@
 		)
 	)
-	(label "AUX_CH2_m"
-		(at 224.79 97.79 180)
-		(fields_autoplaced yes)
-		(effects
-			(font
-				(size 0.889 0.889)
-			)
-			(justify right bottom)
-		)
-	)
 	(label "CH_TPS_m"
 		(at 224.79 105.41 180)
@@
 		)
 	)
-	(label "AUX_CH1_m"
-		(at 224.79 100.33 180)
-		(fields_autoplaced yes)
-		(effects
-			(font
-				(size 0.889 0.889)
-			)
-			(justify right bottom)
-		)
-	)
 	(label "CH_VBATT_m"
 		(at 110.49 52.07 180)
@@
 		)
 	)
-	(label "AUX_CH3_m"
-		(at 224.79 95.25 180)
-		(fields_autoplaced yes)
-		(effects
-			(font
-				(size 0.889 0.889)
-			)
-			(justify right bottom)
-		)
-	)
 	(label "CH_O2_m"
 		(at 92.075 111.76 180)
@@
 		)
 	)
-	(label "AUX_CH8_m"
-		(at 245.11 97.79 0)
-		(fields_autoplaced yes)
-		(effects
-			(font
-				(size 0.889 0.889)
-			)
-			(justify left bottom)
-		)
-	)
 	(label "CH_MAP_m"
 		(at 245.11 102.87 0)
@@
 		)
 	)
-	(label "AUX_CH5_m"
-		(at 224.79 92.71 180)
-		(fields_autoplaced yes)
-		(effects
-			(font
-				(size 0.889 0.889)
-			)
-			(justify right bottom)
-		)
-	)
 	(global_label "TPS_Sensor"
 		(shape input)
@@
 	(global_label "ext_a1_in"
 		(shape input)
+		(at 245.11 97.79 0)
+		(fields_autoplaced yes)
+		(effects
+			(font
+				(size 1.27 1.27)
+			)
+			(justify left)
+		)
+		(property "Intersheetrefs" "${INTERSHEET_REFS}"
+			(at 256.9851 97.79 0)
+			(effects
+				(font
+					(size 1.27 1.27)
+				)
+				(justify left)
+				(hide yes)
+			)
+		)
+	)
+	(global_label "ext_a1_in"
+		(shape input)
 		(at 156.21 109.22 180)
 		(fields_autoplaced yes)
@@
 				(hide yes)
 			)
+		)
+	)
+	(global_label "ext_a0_in"
+		(shape input)
+		(at 245.11 100.33 0)
+		(fields_autoplaced yes)
+		(effects
+			(font
+				(size 1.27 1.27)
+			)
+			(justify left)
+		)
+		(property "Intersheetrefs" "${INTERSHEET_REFS}"
+			(at 256.9851 100.33 0)
+			(effects
+				(font
+					(size 1.27 1.27)
+				)
+				(justify left)
+				(hide yes)
+			)

Commit message: finish pcb layout
Changed lines of the file:
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@@
+	(wire
+		(pts
+			(xy 252.73 41.91) (xy 259.08 41.91)
+		)
+		(stroke
+			(width 0)
+			(type default)
+		)
+	)
 	(wire
 		(pts
@@
 		)
 	)
+	(global_label "ACCL_CS"
+		(shape input)
+		(at 210.82 53.34 180)
+		(fields_autoplaced yes)
+		(effects
+			(font
+				(size 1.27 1.27)
+			)
+			(justify right)
+		)
+		(property "Intersheetrefs" "${INTERSHEET_REFS}"
+			(at 199.731 53.34 0)
+			(effects
+				(font
+					(size 1.27 1.27)
+				)
+				(justify right)
+				(hide yes)
+			)
+		)
+	)
+	(global_label "BARO_CS"
+		(shape input)
+		(at 252.73 41.91 180)
+		(fields_autoplaced yes)
+		(effects
+			(font
+				(size 0.8 0.8)
+			)
+			(justify right)
+		)
+		(property "Intersheetrefs" "${INTERSHEET_REFS}"
+			(at 245.5545 41.91 0)
+			(effects
+				(font
+					(size 1.27 1.27)
+				)
+				(justify right)
+				(hide yes)
+			)
+		)
+	)
 	(global_label "CLT_Sensor"
 		(shape input)
@@
 		)
 	)
-	(hierarchical_label "BARO_CS"
-		(shape input)
-		(at 259.08 41.91 180)
-		(fields_autoplaced yes)
-		(effects
-			(font
-				(size 0.889 0.889)
-			)
-			(justify right)
-		)
-	)
 	(hierarchical_label "SPI2_MOSI"
 		(shape input)
@@
 		(fields_autoplaced yes)
 		(effects
-			(font
-				(size 0.889 0.889)
-			)
-			(justify right)
-		)
-	)
-	(hierarchical_label "ACCL_CS"
-		(shape input)
-		(at 210.82 53.34 180)
-		(fields_autoplaced yes)
-		(effects

Commit message: update SD card holder to Molex 47352
Parts:
- TP10, TP11, TP14, TP15, TP16, TP9: now left out of the parts list
Changed lines of the file:
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@@
 	(version 20231120)
 	(generator "eeschema")
-	(generator_version "7.99")
+	(generator_version "8.0")
 	(paper "A4")
 	(title_block
 		(title "μEFI (Speeduino FW compatible)")
 		(date "2023-12-25")
-		(rev "v6")
+		(rev "v6.1")
 		(company "Churrosoft ®")
-		(comment 1 "CERN-OHL-S-2.0 license\n")
+		(comment 1 "CERN-OHL-S-2.0 license")
 	)
 	(junction
@@
 		(unit 1)
 		(exclude_from_sim no)
-		(in_bom yes)
+		(in_bom no)
 		(on_board yes)
 		(dnp no)
@@
 		(unit 1)
 		(exclude_from_sim no)
-		(in_bom yes)
+		(in_bom no)
 		(on_board yes)
 		(dnp no)
@@
 		(unit 1)
 		(exclude_from_sim no)
-		(in_bom yes)
+		(in_bom no)
 		(on_board yes)
 		(dnp no)
@@
 		(unit 1)
 		(exclude_from_sim no)
-		(in_bom yes)
+		(in_bom no)
 		(on_board yes)
 		(dnp no)
@@
 		(unit 1)
 		(exclude_from_sim no)
-		(in_bom yes)
+		(in_bom no)
 		(on_board yes)
 		(dnp no)
@@
 		(unit 1)
 		(exclude_from_sim no)
-		(in_bom yes)
+		(in_bom no)
 		(on_board yes)
 		(dnp no)

Commit message: update footprints
Parts:
- R18, R19, R20, R28, R29, R30: footprint Resistor_SMD:R_0603_1608Metric -> Resistor_SMD:R_0805_2012Metric
Changed lines of the file:
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@@
 			)
 		)
-		(property "Footprint" "Resistor_SMD:R_0603_1608Metric"
+		(property "Footprint" "Resistor_SMD:R_0805_2012Metric"
 			(at 38.1 35.56 0)
 			(effects
@@
 			)
 		)
-		(property "Footprint" "Resistor_SMD:R_0603_1608Metric"
+		(property "Footprint" "Resistor_SMD:R_0805_2012Metric"
 			(at 38.1 72.39 0)
 			(effects
@@
 			)
 		)
-		(property "Footprint" "Resistor_SMD:R_0603_1608Metric"
+		(property "Footprint" "Resistor_SMD:R_0805_2012Metric"
 			(at 78.74 72.39 0)
 			(effects
@@
 			)
 		)
-		(property "Footprint" "Resistor_SMD:R_0603_1608Metric"
+		(property "Footprint" "Resistor_SMD:R_0805_2012Metric"
 			(at 76.835 111.76 0)
 			(effects
@@
 			)
 		)
-		(property "Footprint" "Resistor_SMD:R_0603_1608Metric"
+		(property "Footprint" "Resistor_SMD:R_0805_2012Metric"
 			(at 79.375 33.02 0)
 			(effects
@@
 			)
 		)
-		(property "Footprint" "Resistor_SMD:R_0603_1608Metric"
+		(property "Footprint" "Resistor_SMD:R_0805_2012Metric"
 			(at 40.64 111.76 0)
 			(effects

Commit message: update from inventree
Parts:
- C11, C12, C13, C21, C22, C23, C47, C50: STOCK (none) -> CAP-000175-00
- C16, C17, C18, C24, C27, C28: STOCK (none) -> CAP-000273-00
- R14, R15, R25: STOCK (none) -> RES-000338-00
- R17, R24, R33, R35, R36, R45, R46, R47: STOCK (none) -> RES-000339-00
- R18, R19, R20, R28, R29, R30: LCSC C23179 -> C114564; STOCK (none) -> RES-000077-00
- R21: STOCK (none) -> RES-000340-00
- R22: STOCK (none) -> RES-000341-00
- R23, R26, R39, R40, R41, R50, R51, R52: STOCK (none) -> RES-000342-00
- TP10, TP11, TP14, TP15, TP16, TP9: now not fitted
- U10: STOCK (none) -> ICS-000357-00
- U21: LCSC (none) -> C579454; STOCK (none) -> ICS-000363-00
- U6, U7: STOCK (none) -> ICS-000346-00
- U9: STOCK (none) -> DIO-000356-00
