File: hw_v1/vr_inputs.kicad_sch (KiCad schematic)
At the start: 32 parts, among them Q1 AO3400A, Q2 AO3400A, SW1 SW_DIP_x02, U4 MAX9926UAEE+

Commit message: add sensors/ relay ouputs, connect all IO to mcu
Other:
- company: (none) -> Churrosoft ®
- title: (none) -> μEFI (Speeduino FW compatible)
Changed lines of the file:
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@@
 	(generator_version "7.99")
 	(paper "A4")
+	(title_block
+		(title "μEFI (Speeduino FW compatible)")
+		(date "2023-12-25")
+		(rev "v6")
+		(company "Churrosoft ®")
+		(comment 1 "CERN-OHL-S-2.0 license\n")
+	)
 	(junction
 		(at 179.705 73.66)

Commit message: wip pcb layout
Parts:
- removed SW1: SW_DIP_x02, Button_Switch_SMD:SW_DIP_SPSTx02_Slide_6.7x6.64mm_W8.61mm_P2.54mm_LowProfile, symbol Switch:SW_DIP_x02
- added JP11, JP12: Jumper_2_Open, Jumper:SolderJumper-2_P1.3mm_Open_RoundedPad1.0x1.5mm, symbol Jumper:Jumper_2_Open
Connections:
- net GND: now also JP11.1 (A), JP12.1 (A)
- net at C8.2: now also JP12.2 (B)
- net at C7.2: now also JP11.2 (B)
Changed lines of the file:
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@@
 	(wire
 		(pts
-			(xy 135.89 162.56) (xy 135.89 165.1)
+			(xy 135.89 162.56) (xy 135.89 167.64)
 		)
 		(stroke
@@
 	(wire
 		(pts
+			(xy 135.89 177.8) (xy 135.89 180.34)
+		)
+		(stroke
+			(width 0)
+			(type default)
+		)
+	)
+	(wire
+		(pts
 			(xy 60.96 121.285) (xy 60.96 124.46)
 		)
@@
 	(wire
 		(pts
-			(xy 138.43 162.56) (xy 138.43 165.1)
+			(xy 138.43 162.56) (xy 138.43 167.64)
 		)
 		(stroke
@@
 		(pts
 			(xy 134.62 157.48) (xy 134.62 153.67)
+		)
+		(stroke
+			(width 0)
+			(type default)
+		)
+	)
+	(wire
+		(pts
+			(xy 138.43 177.8) (xy 138.43 180.34)
 		)
 		(stroke
@@
 	)
 	(symbol
+		(lib_id "Jumper:Jumper_2_Open")
+		(at 138.43 172.72 90)
+		(unit 1)
+		(exclude_from_sim no)
+		(in_bom yes)
+		(on_board yes)
+		(dnp no)
+		(fields_autoplaced yes)
+		(property "Reference" "JP12"
+			(at 139.7 171.4499 90)
+			(effects
+				(font
+					(size 1.27 1.27)
+				)
+				(justify right)
+				(hide yes)
+			)
+		)
+		(property "Value" "Jumper_2_Open"
+			(at 139.7 173.9899 90)
+			(effects
+				(font
+					(size 1.27 1.27)
+				)
+				(justify right)
+				(hide yes)
+			)
+		)
+		(property "Footprint" "Jumper:SolderJumper-2_P1.3mm_Open_RoundedPad1.0x1.5mm"
+			(at 138.43 172.72 0)
+			(effects
+				(font
+					(size 1.27 1.27)
+				)
+				(hide yes)
+			)
+		)
+		(property "Datasheet" "~"
+			(at 138.43 172.72 0)
+			(effects
+				(font
+					(size 1.27 1.27)
+				)
+				(hide yes)
+			)
+		)
+		(property "Description" "Jumper, 2-pole, open"
+			(at 138.43 172.72 0)
+			(effects
+				(font
+					(size 1.27 1.27)
+				)
+				(hide yes)
+			)
+		)
+		(pin "2"
+		)
+		(pin "1"
+		)
+		(instances
+			(project "hw_v1"
+				(path "/b3feb07e-be80-40e1-bd13-6cd54c2f8b0c/27977e95-ecc9-4124-9dfb-b7b6f545e8f2"
+					(reference "JP12")
+					(unit 1)
+				)
+			)
+		)
+	)
+	(symbol
 		(lib_id "Jumper:Jumper_3_Bridged12")
 		(at 78.105 136.525 0)
@@
 	)
 	(symbol
-		(lib_id "Switch:SW_DIP_x02")
-		(at 138.43 172.72 90)
-		(unit 1)
-		(exclude_from_sim no)
-		(in_bom yes)
-		(on_board yes)
-		(dnp no)
-		(fields_autoplaced yes)
-		(property "Reference" "SW1"
-			(at 142.24 171.45 90)
-			(effects
-				(font
-					(size 1.27 1.27)
-				)
-				(justify right)
-			)
-		)
-		(property "Value" "SW_DIP_x02"
-			(at 142.24 173.99 90)
-			(effects
-				(font
-					(size 1.27 1.27)
-				)
-				(justify right)
-			)
-		)
-		(property "Footprint" "Button_Switch_SMD:SW_DIP_SPSTx02_Slide_6.7x6.64mm_W8.61mm_P2.54mm_LowProfile"
-			(at 138.43 172.72 0)
-			(effects
-				(font
-					(size 1.27 1.27)
-				)
-				(hide yes)
-			)
-		)
-		(property "Datasheet" "~"
-			(at 138.43 172.72 0)
-			(effects
-				(font
-					(size 1.27 1.27)
-				)
-				(hide yes)
-			)
-		)
-		(property "Description" ""
-			(at 138.43 172.72 0)
-			(effects
-				(font
-					(size 1.27 1.27)
-				)
-				(hide yes)
-			)
-		)
-		(pin "1"
-		)
-		(pin "2"
-		)
-		(pin "3"
-		)
-		(pin "4"
-		)
-		(instances
-			(project "hw_v1"
-				(path "/b3feb07e-be80-40e1-bd13-6cd54c2f8b0c/27977e95-ecc9-4124-9dfb-b7b6f545e8f2"
-					(reference "SW1")
-					(unit 1)
-				)
-			)
-		)
-	)
-	(symbol
 		(lib_id "Device:R")
 		(at 73.66 29.21 90)
@@
 					(unit 1)
 				)
+			)
+		)
+	)
+	(symbol
+		(lib_id "Jumper:Jumper_2_Open")
+		(at 135.89 172.72 90)
+		(unit 1)
+		(exclude_from_sim no)
+		(in_bom yes)
+		(on_board yes)
+		(dnp no)
+		(fields_autoplaced yes)
+		(property "Reference" "JP11"
+			(at 137.16 171.4499 90)
+			(effects
+				(font
+					(size 1.27 1.27)
+				)
+				(justify right)
+				(hide yes)
+			)
+		)
+		(property "Value" "Jumper_2_Open"
+			(at 137.16 173.9899 90)
+			(effects
+				(font
+					(size 1.27 1.27)
+				)
+				(justify right)
+				(hide yes)
+			)
+		)
+		(property "Footprint" "Jumper:SolderJumper-2_P1.3mm_Open_RoundedPad1.0x1.5mm"
+			(at 135.89 172.72 0)
+			(effects
+				(font
+					(size 1.27 1.27)
+				)
+				(hide yes)
+			)
+		)
+		(property "Datasheet" "~"
+			(at 135.89 172.72 0)
+			(effects
+				(font
+					(size 1.27 1.27)
+				)
+				(hide yes)
+			)
+		)
+		(property "Description" "Jumper, 2-pole, open"
+			(at 135.89 172.72 0)
+			(effects
+				(font
+					(size 1.27 1.27)
+				)
+				(hide yes)
+			)
+		)
+		(pin "2"
+		)
+		(pin "1"
+		)
+		(instances
+			(project "hw_v1"
+				(path "/b3feb07e-be80-40e1-bd13-6cd54c2f8b0c/27977e95-ecc9-4124-9dfb-b7b6f545e8f2"
+					(reference "JP11")
+					(unit 1)
+				)

Commit message: wip sensors pcb layout
Other:
- note added: "Todos usan de 1/4 - 1/8w, revisar"
Changed lines of the file:
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@@
+		)
+	)
+	(polyline
+		(pts
+			(xy 74.93 45.72) (xy 74.93 39.37)
+		)
+		(stroke
+			(width 0)
+			(type default)
 		)
 	)
@@
 		)
 	)
+	(polyline
+		(pts
+			(xy 15.24 39.37) (xy 74.93 39.37)
+		)
+		(stroke
+			(width 0)
+			(type default)
+		)
+	)
 	(wire
 		(pts
@@
 		)
 	)
+	(text "Todos usan de 1/4 - 1/8w, revisar"
+		(exclude_from_sim no)
+		(at 32.512 41.656 0)
+		(effects
+			(font
+				(size 1.27 1.27)
+			)
+		)
+	)

Commit message: placed al SMD, wip pmic traces
Parts:
- R2, R3, R4, R5, R7, R8: footprint Resistor_SMD:R_1210_3225Metric -> Resistor_SMD:R_0805_2012Metric
Connections:
- net CKP+ renamed CRANK+
- net CKP- renamed CRANK-
- net CMP+ renamed CAM+
- net CMP- renamed CAM-
Changed lines of the file:
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@@
 	)
 	(junction
+		(at 62.357 93.345)
+		(diameter 0)
+		(color 0 0 0 0)
+	)
+	(junction
 		(at 88.265 93.345)
 		(diameter 1.016)
@@
 	)
 	(junction
+		(at 62.23 67.31)
+		(diameter 0)
+		(color 0 0 0 0)
+	)
+	(junction
 		(at 139.7 153.67)
 		(diameter 0)
@@
 	)
 	(junction
-		(at 61.595 93.345)
-		(diameter 1.016)
-		(color 0 0 0 0)
-	)
-	(junction
 		(at 114.3 73.66)
 		(diameter 1.016)
@@
 	(wire
 		(pts
+			(xy 62.23 67.31) (xy 62.23 69.85)
+		)
+		(stroke
+			(width 0)
+			(type solid)
+		)
+	)
+	(wire
+		(pts
 			(xy 102.87 86.36) (xy 102.87 93.345)
 		)
@@
 	(wire
 		(pts
+			(xy 62.357 93.345) (xy 61.595 93.345)
+		)
+		(stroke
+			(width 0)
+			(type solid)
+		)
+	)
+	(wire
+		(pts
 			(xy 135.89 177.8) (xy 135.89 180.34)
 		)
@@
 	(wire
 		(pts
-			(xy 61.595 93.345) (xy 64.77 93.345)
+			(xy 62.357 93.345) (xy 64.77 93.345)
 		)
 		(stroke
@@
 	(wire
 		(pts
-			(xy 61.595 92.964) (xy 61.595 93.345)
+			(xy 62.357 92.71) (xy 62.357 93.345)
 		)
 		(stroke
@@
 	(wire
 		(pts
+			(xy 57.15 67.31) (xy 62.23 67.31)
+		)
+		(stroke
+			(width 0)
+			(type default)
+		)
+	)
+	(wire
+		(pts
 			(xy 110.49 46.99) (xy 98.425 46.99)
 		)
@@
 	(wire
 		(pts
-			(xy 56.388 92.964) (xy 61.595 92.964)
-		)
-		(stroke
-			(width 0)
-			(type solid)
-		)
-	)
-	(wire
-		(pts
-			(xy 62.23 69.85) (xy 62.23 67.31)
+			(xy 57.15 92.71) (xy 62.357 92.71)
 		)
 		(stroke
@@
 		)
 	)
-	(global_label "CKP+"
+	(global_label "CAM+"
 		(shape input)
-		(at 73.025 142.24 180)
+		(at 41.91 50.8 180)
 		(effects
 			(font
@@
 		)
 		(property "Intersheetrefs" "${INTERSHEET_REFS}"
-			(at 65.2295 142.1606 0)
+			(at 41.91 50.8 0)
 			(effects
 				(font
 					(size 1.27 1.27)
 				)
-				(justify right)
 				(hide yes)
 			)
 		)
 	)
-	(global_label "CKP-"
+	(global_label "CAM-"
 		(shape input)
-		(at 56.388 92.964 180)
+		(at 57.15 67.31 180)
 		(effects
 			(font
@@
 		)
 		(property "Intersheetrefs" "${INTERSHEET_REFS}"
-			(at 48.5925 92.8846 0)
+			(at 57.15 67.31 0)
 			(effects
 				(font
 					(size 1.27 1.27)
 				)
-				(justify right)
 				(hide yes)
 			)
 		)
 	)
-	(global_label "CMP+"
+	(global_label "CRANK+"
 		(shape input)
-		(at 41.91 50.8 180)
+		(at 73.66 142.24 180)
 		(effects
 			(font
@@
 		)
 		(property "Intersheetrefs" "${INTERSHEET_REFS}"
-			(at 33.9331 50.7206 0)
+			(at 73.66 142.24 0)
 			(effects
 				(font
 					(size 1.27 1.27)
 				)
-				(justify right)
 				(hide yes)
 			)
 		)
 	)
-	(global_label "CMP-"
+	(global_label "CRANK-"
 		(shape input)
-		(at 62.23 67.31 180)
+		(at 57.15 92.71 180)
 		(effects
 			(font
@@
 		)
 		(property "Intersheetrefs" "${INTERSHEET_REFS}"
-			(at 54.2531 67.2306 0)
+			(at 57.15 92.71 0)
 			(effects
 				(font
 					(size 1.27 1.27)
 				)
-				(justify right)
 				(hide yes)
 			)
@@
 			)
 		)
-		(property "Footprint" "Resistor_SMD:R_1210_3225Metric"
+		(property "Footprint" "Resistor_SMD:R_0805_2012Metric"
 			(at 89.535 52.705 0)
 			(effects
@@
 			)
 		)
-		(property "Footprint" "Resistor_SMD:R_1210_3225Metric"
+		(property "Footprint" "Resistor_SMD:R_0805_2012Metric"
 			(at 68.58 46.99 0)
 			(effects
@@
 			)
 		)
-		(property "Footprint" "Resistor_SMD:R_1210_3225Metric"
+		(property "Footprint" "Resistor_SMD:R_0805_2012Metric"
 			(at 67.31 113.665 0)
 			(effects
@@
 			)
 		)
-		(property "Footprint" "Resistor_SMD:R_1210_3225Metric"
+		(property "Footprint" "Resistor_SMD:R_0805_2012Metric"
 			(at 88.265 99.06 0)
 			(effects
@@
 			)
 		)
-		(property "Footprint" "Resistor_SMD:R_1210_3225Metric"
+		(property "Footprint" "Resistor_SMD:R_0805_2012Metric"
 			(at 67.31 93.345 0)
 			(effects
@@
 			)
 		)
-		(property "Footprint" "Resistor_SMD:R_1210_3225Metric"
+		(property "Footprint" "Resistor_SMD:R_0805_2012Metric"
 			(at 68.58 67.31 0)
 			(effects

Commit message: update SD card holder to Molex 47352
Parts:
- JP1, JP11, JP12, JP2, JP3, JP4, TP1, TP2, TP3, TP4, TP5, TP6, U4: now left out of the parts list
Changed lines of the file:
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@@
 	(version 20231120)
 	(generator "eeschema")
-	(generator_version "7.99")
+	(generator_version "8.0")
 	(paper "A4")
 	(title_block
 		(title "μEFI (Speeduino FW compatible)")
 		(date "2023-12-25")
-		(rev "v6")
+		(rev "v6.1")
 		(company "Churrosoft ®")
-		(comment 1 "CERN-OHL-S-2.0 license\n")
+		(comment 1 "CERN-OHL-S-2.0 license")
 	)
 	(junction
@@
 		(unit 1)
 		(exclude_from_sim no)
-		(in_bom yes)
+		(in_bom no)
 		(on_board yes)
 		(dnp no)
@@
 		(unit 1)
 		(exclude_from_sim no)
-		(in_bom yes)
+		(in_bom no)
 		(on_board yes)
 		(dnp no)
@@
 		(unit 1)
 		(exclude_from_sim no)
-		(in_bom yes)
+		(in_bom no)
 		(on_board yes)
 		(dnp no)
@@
 		(unit 1)
 		(exclude_from_sim no)
-		(in_bom yes)
+		(in_bom no)
 		(on_board yes)
 		(dnp no)
@@
 		(unit 1)
 		(exclude_from_sim no)
-		(in_bom yes)
+		(in_bom no)
 		(on_board yes)
 		(dnp no)
@@
 		(unit 1)
 		(exclude_from_sim no)
-		(in_bom yes)
+		(in_bom no)
 		(on_board yes)
 		(dnp no)
@@
 		(unit 1)
 		(exclude_from_sim no)
-		(in_bom yes)
+		(in_bom no)
 		(on_board yes)
 		(dnp no)
@@
 		(unit 1)
 		(exclude_from_sim no)
-		(in_bom yes)
+		(in_bom no)
 		(on_board yes)
 		(dnp no)
@@
 		(unit 1)
 		(exclude_from_sim no)
-		(in_bom yes)
+		(in_bom no)
 		(on_board yes)
 		(dnp no)
@@
 		(unit 1)
 		(exclude_from_sim no)
-		(in_bom yes)
+		(in_bom no)
 		(on_board yes)
 		(dnp no)
@@
 		(unit 1)
 		(exclude_from_sim no)
-		(in_bom yes)
+		(in_bom no)
 		(on_board yes)
 		(dnp no)
@@
 		(unit 1)
 		(exclude_from_sim no)
-		(in_bom yes)
+		(in_bom no)
 		(on_board yes)
 		(dnp no)
@@
 		(unit 1)
 		(exclude_from_sim no)
-		(in_bom yes)
+		(in_bom no)
 		(on_board yes)
 		(dnp no)

Commit message: update vr inputs
Parts:
- C8: value 4700pF -> 4.7nF; LCSC C576950 -> C106218
Changed lines of the file:
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@@
 			)
 		)
-		(property "Value" "4700pF"
-			(at 142.0242 161.1693 0)
+		(property "Value" "4.7nF"
+			(at 141.986 161.29 0)
 			(effects
 				(font
@@
 			)
 		)
-		(property "LCSC" "C576950"
+		(property "LCSC" "C106218"
 			(at 139.7 160.02 0)
 			(effects

Commit message: update footprints
Parts:
- R2, R3, R4, R5: value 10K 1/2W -> 10k; footprint Resistor_SMD:R_0805_2012Metric -> Resistor_SMD:R_0603_1608Metric; LCSC C2974059 -> C115324
Changed lines of the file:
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@@
 			)
 		)
-		(property "Value" "10K 1/2W"
+		(property "Value" "10k"
 			(at 68.58 44.3419 90)
 			(effects
@@
 			)
 		)
-		(property "Footprint" "Resistor_SMD:R_0805_2012Metric"
+		(property "Footprint" "Resistor_SMD:R_0603_1608Metric"
 			(at 68.58 46.99 0)
 			(effects
@@
 			)
 		)
-		(property "LCSC" "C2974059"
+		(property "LCSC" "C115324"
 			(at 68.58 46.99 90)
 			(effects
@@
 			)
 		)
-		(property "Value" "10K 1/2W"
+		(property "Value" "10k"
 			(at 67.31 111.0169 90)
 			(effects
@@
 			)
 		)
-		(property "Footprint" "Resistor_SMD:R_0805_2012Metric"
+		(property "Footprint" "Resistor_SMD:R_0603_1608Metric"
 			(at 67.31 113.665 0)
 			(effects
@@
 			)
 		)
-		(property "LCSC" "C2974059"
+		(property "LCSC" "C115324"
 			(at 67.31 113.665 90)
 			(effects
@@
 			)
 		)
-		(property "Value" "10K 1/2W"
+		(property "Value" "10k"
 			(at 67.31 90.6969 90)
 			(effects
@@
 			)
 		)
-		(property "Footprint" "Resistor_SMD:R_0805_2012Metric"
+		(property "Footprint" "Resistor_SMD:R_0603_1608Metric"
 			(at 67.31 93.345 0)
 			(effects
@@
 			)
 		)
-		(property "LCSC" "C2974059"
+		(property "LCSC" "C115324"
 			(at 67.31 93.345 90)
 			(effects
@@
 			)
 		)
-		(property "Value" "10K 1/2W"
+		(property "Value" "10k"
 			(at 68.58 64.6619 90)
 			(effects
@@
 			)
 		)
-		(property "Footprint" "Resistor_SMD:R_0805_2012Metric"
+		(property "Footprint" "Resistor_SMD:R_0603_1608Metric"
 			(at 68.58 67.31 0)
 			(effects
@@
 			)
 		)
-		(property "LCSC" "C2974059"
+		(property "LCSC" "C115324"
 			(at 68.58 67.31 90)
 			(effects

Commit message: update from inventree
Parts:
- C1, C2, C3, C4, C5, C6, C7: STOCK (none) -> CAP-000323-00
- C8: STOCK (none) -> CAP-000324-00
- JP1, JP11, JP12, JP2, JP3, JP4, TP1, TP2, TP3, TP4, TP5, TP6: now not fitted
- Q1, Q2: STOCK (none) -> TRA-000186-00
- R10, R11: LCSC C25804 -> C115324; STOCK (none) -> RES-000118-00
- R2, R3, R4, R5: STOCK (none) -> RES-000118-00
- R6, R9: STOCK (none) -> RES-000107-00
- R7, R8: LCSC C407178 -> C2933454; STOCK (none) -> RES-000337-00
- U4: LCSC (none) -> -; STOCK (none) -> ICS-000034-00
Changed lines of the file:
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@@
 			)
 		)
+		(property "STOCK" "CAP-000323-00"
+			(at 60.96 118.745 0)
+			(effects
+				(font
+					(size 1.27 1.27)
+				)
+				(hide yes)
+			)
+		)
 		(pin "1"
 		)
@@
 			)
 		)
+		(property "STOCK" "CAP-000324-00"
+			(at 139.7 160.02 0)
+			(effects
+				(font
+					(size 1.27 1.27)
+				)
+				(hide yes)
+			)
+		)
 		(pin "1"
 		)
@@
 			)
 		)
+		(property "STOCK" "RES-000107-00"
+			(at 100.965 128.905 0)
+			(effects
+				(font
+					(size 1.27 1.27)
+				)
+				(hide yes)
+			)
+		)
 		(pin "1"
 		)
@@
 			)
 		)
+		(property "STOCK" "TRA-000186-00"
+			(at 68.58 34.29 0)
+			(effects
+				(font
+					(size 1.27 1.27)
+				)
+				(hide yes)
+			)
+		)
 		(pin "1"
 		)
@@
 			)
 		)
+		(property "STOCK" "CAP-000323-00"
+			(at 98.425 55.245 0)
+			(effects
+				(font
+					(size 1.27 1.27)
+				)
+				(hide yes)
+			)
+		)
 		(pin "1"
 		)
@@
 			)
 		)
+		(property "STOCK" "TRA-000186-00"
+			(at 95.885 133.985 0)
+			(effects
+				(font
+					(size 1.27 1.27)
+				)
+				(hide yes)
+			)
+		)
 		(pin "1"
 		)
@@
 		(in_bom no)
 		(on_board yes)
-		(dnp no)
+		(dnp yes)
 		(fields_autoplaced yes)
 		(property "Reference" "JP12"
@@
 		(in_bom no)
 		(on_board yes)
-		(dnp no)
+		(dnp yes)
 		(property "Reference" "JP2"
 			(at 76.835 133.985 90)
@@
 		(in_bom no)
 		(on_board yes)
-		(dnp no)
+		(dnp yes)
 		(property "Reference" "JP4"
 			(at 91.6687 60.4456 90)
@@
 			)
 		)
-		(property "LCSC" "C407178"
+		(property "LCSC" "C2933454"
 			(at 89.535 52.705 90)
 			(effects
@@
 			)
 		)
+		(property "STOCK" "RES-000337-00"
+			(at 89.535 52.705 0)
+			(effects
+				(font
+					(size 1.27 1.27)
+				)
+				(hide yes)
+			)
+		)
 		(pin "1"
 		)
@@
 			)
 		)
+		(property "STOCK" "CAP-000323-00"
+			(at 62.23 72.39 0)
+			(effects
+				(font
+					(size 1.27 1.27)
+				)
+				(hide yes)
+			)
+		)
 		(pin "1"
 		)
@@
 		(in_bom no)
 		(on_board yes)
-		(dnp no)
+		(dnp yes)
 		(property "Reference" "TP1"
 			(at 99.06 90.8684 0)
@@
 		(in_bom no)
 		(on_board yes)
-		(dnp no)
+		(dnp yes)
 		(property "Reference" "TP2"
 			(at 100.33 44.5134 0)
@@
 			)
 		)
+		(property "STOCK" "CAP-000323-00"
+			(at 97.155 101.6 0)
+			(effects
+				(font
+					(size 1.27 1.27)
+				)
+				(hide yes)
+			)
+		)
 		(pin "1"
 		)
@@
 			)
 		)
+		(property "STOCK" "RES-000107-00"
+			(at 73.66 29.21 0)
+			(effects
+				(font
+					(size 1.27 1.27)
+				)
+				(hide yes)
+			)
+		)
 		(pin "1"
 		)
@@
 			)
 		)
+		(property "STOCK" "RES-000118-00"
+			(at 68.58 46.99 0)
+			(effects
+				(font
+					(size 1.27 1.27)
+				)
+				(hide yes)
+			)
+		)
 		(pin "1"
 		)
@@
 			)
 		)
+		(property "STOCK" "RES-000118-00"
+			(at 67.31 113.665 0)
+			(effects
+				(font
+					(size 1.27 1.27)
+				)
+				(hide yes)
+			)
+		)
 		(pin "1"
 		)
@@
 		(in_bom no)
 		(on_board yes)
-		(dnp no)
+		(dnp yes)
 		(property "Reference" "JP3"
 			(at 90.3987 106.8006 90)
@@
 			)
 		)
+		(property "STOCK" "CAP-000323-00"
+			(at 62.865 52.07 0)
+			(effects
+				(font
+					(size 1.27 1.27)
+				)
+				(hide yes)
+			)
+		)
 		(pin "1"
 		)
@@
 		(in_bom no)
 		(on_board yes)
-		(dnp no)
+		(dnp yes)
 		(fields_autoplaced yes)
 		(property "Reference" "JP11"
@@
 			)
 		)
+		(property "STOCK" "CAP-000323-00"
+			(at 134.62 160.02 0)
+			(effects
+				(font
+					(size 1.27 1.27)
+				)
+				(hide yes)
+			)
+		)
 		(pin "1"
 		)
@@
 		(in_bom no)
 		(on_board yes)
-		(dnp no)
+		(dnp yes)
 		(property "Reference" "JP1"
 			(at 48.26 44.45 90)
@@
 			)
 		)
-		(property "LCSC" "C25804"
+		(property "LCSC" "C115324"
 			(at 164.0587 67.4306 0)
 			(effects
@@
 			)
 		)
+		(property "STOCK" "RES-000118-00"
+			(at 162.56 68.58 0)
+			(effects
+				(font
+					(size 1.27 1.27)
+				)
+				(hide yes)
+			)
+		)
 		(pin "1"
 		)
@@
 		(in_bom no)
 		(on_board yes)
-		(dnp no)
+		(dnp yes)
 		(property "Reference" "TP5"
 			(at 177.8 76.1366 0)
@@
 			)
 		)
-		(property "LCSC" "C25804"
+		(property "LCSC" "C115324"
 			(at 175.4887 69.9706 0)
 			(effects
@@
 			)
 		)
+		(property "STOCK" "RES-000118-00"
+			(at 173.99 71.12 0)
+			(effects
+				(font
+					(size 1.27 1.27)
+				)
+				(hide yes)
+			)
+		)
 		(pin "1"
 		)
@@
 		(in_bom no)
 		(on_board yes)
-		(dnp no)
+		(dnp yes)
 		(property "Reference" "TP6"
 			(at 182.245 68.6434 0)
@@
 		(in_bom no)
 		(on_board yes)
-		(dnp no)
+		(dnp yes)
 		(property "Reference" "TP3"
 			(at 96.52 69.7866 0)
@@
 			)
 		)
-		(property "LCSC" "C407178"
+		(property "LCSC" "C2933454"
 			(at 88.265 99.06 90)
 			(effects
@@
 			)
 		)
+		(property "STOCK" "RES-000337-00"
+			(at 88.265 99.06 0)
+			(effects
+				(font
+					(size 1.27 1.27)
+				)
+				(hide yes)
+			)
+		)
 		(pin "1"
 		)
@@
 			)
 		)
+		(property "LCSC" "-"
+			(at 135.89 86.36 0)
+			(effects
+				(font
+					(size 1.27 1.27)
+				)
+				(hide yes)
+			)
+		)
+		(property "STOCK" "ICS-000034-00"
+			(at 135.89 86.36 0)
+			(effects
+				(font
+					(size 1.27 1.27)
+				)
+				(hide yes)
+			)
+		)
 		(pin "1"
 		)
@@
 		(in_bom no)
 		(on_board yes)
-		(dnp no)
+		(dnp yes)
 		(property "Reference" "TP4"
 			(at 104.775 116.1416 0)
@@
 			)
 		)
+		(property "STOCK" "RES-000118-00"
+			(at 67.31 93.345 0)
+			(effects
+				(font
+					(size 1.27 1.27)
+				)
+				(hide yes)
+			)
+		)
 		(pin "1"
 		)
@@
 			)
 		)
+		(property "STOCK" "CAP-000323-00"
+			(at 61.595 98.425 0)
+			(effects
+				(font
+					(size 1.27 1.27)
+				)
+				(hide yes)
+			)
+		)
 		(pin "1"
 		)
@@
 			(effects
 				(font
+					(size 1.27 1.27)
+				)
+				(hide yes)
+			)
+		)
+		(property "STOCK" "RES-000118-00"
+			(at 68.58 67.31 0)
+			(effects
+				(font
