File: hw_v1/connector.kicad_sch (KiCad schematic)
At the start: 41 parts, among them J1 Conn_02x24_Counter_Clockwise, J12 Delphi_Sicma_24, J13 Delphi_Sicma_24, J14 Conn_01x04, Q3 FDS6890A, U11 L78M05ABDT-TR, U12 LM74800, U19 L78M05ABDT-TR, U8 AMS1117-3.3

Commit message: update from inventree
Parts:
- C14, C49, C9: STOCK (none) -> CAP-000175-00
- C15, C48: STOCK (none) -> CAP-000326-00
- C51, C52, C53: LCSC (none) -> C49678; STOCK (none) -> CAP-000175-00
- C54: LCSC (none) -> C83170; STOCK (none) -> CAP-000072-00
- C55: STOCK (none) -> CAP-000179-00
- D27, D31, D32, D33, D34: STOCK (none) -> DIO-000331-00
- D35: LCSC (none) -> C7436536; STOCK (none) -> DIO-000333-00
- J12, J13, J14, JP10, JP14, JP9, TP19, TP20: now not fitted
- Q3: STOCK (none) -> TRA-000336-00
- R48, R49, R59, R60, R61, R66: STOCK (none) -> RES-000107-00
- R62: LCSC C21190 -> C2933226; STOCK (none) -> RES-000347-00
- R63: LCSC C21190 -> C5126245; STOCK (none) -> RES-000348-00
- R64: LCSC C21190 -> C2930134; STOCK (none) -> RES-000350-00
- R65: LCSC C21190 -> C2998120; STOCK (none) -> RES-000351-00
- R67: LCSC C21190 -> C2906981; STOCK (none) -> RES-000352-00
- U11, U19: STOCK (none) -> PWR-000358-00
- U12: LCSC (none) -> -; STOCK (none) -> DIO-000416-00
- U8: LCSC (none) -> C2992570; STOCK (none) -> PWR-000102-00

Commit message: wip v7
Connections:
- net +12VA: no longer J13.A1
- net +5VA: no longer J13.A3
- net BOOST-OUT: no longer J12.C1
- net CAM+: no longer J13.B1
- net CAM-: no longer J13.B2
- net CAN+: no longer J13.A6
- net CAN-: no longer J13.A7
- net CEL-OUT: no longer J1.28 (Pin_28), J13.A4
- net CLT_Sensor: no longer J13.C5
- net CRANK+: no longer J13.B3
- net CRANK-: no longer J13.B4
- net Clutch_in: no longer J13.A5
- net FAN-OUT: no longer J12.B5
- net FUELPUMP-OUT: no longer J12.C3
- net GND: no longer J13.A2
- net GNDREF: no longer J13.C1
- net IAT_Sensor: no longer J13.C6
- net IDLE-OUT: no longer J12.C2
- net IGN-1-OUT: no longer J12.A5
- net IGN-2-OUT: no longer J12.A6
- net IGN-3-OUT: no longer J12.A7
- net IGN-4-OUT: no longer J12.A8
- net INJ-1-OUT: no longer J12.A1
- net INJ-2-OUT: no longer J12.A2
- net INJ-3-OUT: no longer J12.A3
- net INJ-4-OUT: no longer J12.A4
- net MAP_Sensor: no longer J13.C8
- net O2_Sensor: no longer J13.C4
- net SPARE1_Sensor: no longer J13.C2
- net SPARE2_Sensor: no longer J13.C3
- net STEPPER-A1: no longer J12.B3
- net STEPPER-A2: no longer J12.B4
- net STEPPER-B1: no longer J12.B2
- net STEPPER-B2: no longer J12.B1
- net SW_AC: no longer J13.B8
- net SW_SHIFT: no longer J13.B7
- net SW_TABLE: no longer J13.B6
- net SW_USER: no longer J13.B5
- net TACHO-OUT: no longer J12.B8
- net TPS_Sensor: no longer J13.C7
- new net PROTO-5: J1.28 (Pin_28), J13.A4
Other:
- moved on the sheet: J1, J12, J13
