File: hw_v2/hw_v1.kicad_pcb (KiCad board)
At the start: 4 copper layers, 80.6 x 93.7 mm, 187 parts, among them J1 Conn_02x24_Counter_Clockwise, J14 Conn_01x04, J16 47352-1001, J8 USB_B, J9 Tag connect, SW1 SW_Push, SW2 SW_Push, U1 MAX9924UAUB_, U10 BMP280, U11 L78M05ABDT-TR, U12 VNLD5160TR-E, U13 STM32F407VGTx, U14 TJA1051T-3, U15 25Q16, U16 REF3033, U17 SRV05-4, U18 VNLD5090, U19 L78M05ABDT-TR, U2 TC4424A, U20 VNLD5160TR-E, U21 ADXL343, U23 MCP6004, U24 MCP6004, U25 74LVC2G17, U26 74LVC2G17, U3 TC4424A, U5 TPL7407LAPWR, U6 TJA1051T-3, U7 74LVC2G17, U8 AMS1117-3.3, U9 74LVC2G17, Y1 32.768kHz, Y2 25MHz

Commit message: Fix some ERC errors
Parts:
- moved C38 109.2 mm to (94.6, 104.1), turned to -45 degrees
- moved C37 106.2 mm to (97.7, 100.8), turned to 135 degrees
- moved C36 105.5 mm to (93.3, 111.1), turned to -135 degrees
- moved C26 102.4 mm to (102.1, 121.2), turned to -45 degrees
- moved C35 100.1 mm to (105.9, 121.8)
- moved C33 91.7 mm to (106.5, 97.8), turned to 45 degrees
- moved R27 82.3 mm to (110.6, 100.1), turned to 45 degrees
- moved C29 82.0 mm to (117.2, 109.9), turned to 45 degrees
- moved C31 78.5 mm to (118.6, 111.3), turned to 45 degrees
- moved SW1 18.3 mm to (118.0, 99.0)
- moved SW2 9.18 mm to (129.0, 117.5)
Routing:
- net +3V3: track 0.00 -> 6.93 mm
- net Net-(U13-VCAP_2): track 0.00 -> 4.95 mm
- net Net-(U13-VCAP_1): track 0.00 -> 2.57 mm
Other:
- board text added: "BOOT"
- board text added: "RESET"

Commit message: planito mas catolico
Parts:
- removed R5, R6, R8, R9: 4.7k, Resistor_SMD:R_0603_1608Metric
- removed RN3: 47k, Resistor_SMD:R_Array_Convex_4x0603
- removed U12, U20: VNLD5160TR-E, Package_SO:SOIC-8_3.9x4.9mm_P1.27mm
- removed U2, U3: TC4424A, Package_SO:SOIC-8_3.9x4.9mm_P1.27mm
- removed U9: 74LVC2G17, Package_TO_SOT_SMD:SOT-363_SC-70-6
- added J8: USB_B_Micro, Connector_USB:USB_Mini-B_Tensility_54-00023_Vertical, F.Cu at (2.83, 21.7)
- added U22: STM32F407VGTx, Package_QFP:LQFP-100_14x14mm_P0.5mm, F.Cu at (8.74, 8.74)
- D18: footprint Diode_SMD:D_SOD-323_HandSoldering -> Diode_SMD:D_SOD-323
- J8: value USB_B -> USB_B_Micro
- U1: footprint Package_SO:MSOP-10_3x3mm_P0.5mm -> hw_v2lib:SOP50P490X110-10N
- U14: footprint Package_SO:SOP-8_3.9x4.9mm_P1.27mm -> Package_SO:SOIC-8_3.9x4.9mm_P1.27mm
- moved U1 81.7 mm to (127.5, 105.0)
Connections:
- BT1 pad 1: Net-(BT1-+) -> +BATT
- C26 pad 1: Net-(U13-VCAP_1) -> Net-(U22-VCAP_1)
- C29 pad 1: Net-(U13-VCAP_2) -> Net-(U22-VCAP_2)
- C30 pad 1: GND -> /NRST
- C30 pad 2: /NRST -> GND
- C6 pad 2: Net-(U13-BOOT0) -> Net-(U22-BOOT0)
- D18 pad 1: Net-(BT1-+) -> +BATT
- J1 pad 22: GNDREF -> GND
- J1 pad 27: SPARE2_out -> unconnected-(J1-Pin_27-Pad27)
- J1 pad 28: SPARE1_out -> unconnected-(J1-Pin_28-Pad28)
- J1 pad 37: STEP-B2 -> STEPPER-B2
- J1 pad 38: STEP-B1 -> STEPPER-B1
- J1 pad 39: STEP-A1 -> STEPPER-A2
- J1 pad 40: STEP-A2 -> STEPPER-A1
- J8 pad 4: GND -> unconnected-(J8-ID-Pad4)
- J8 pad 6: (no net) -> GND
- R10 pad 1: Net-(U13-PB2) -> Net-(U22-PB2)
- R27 pad 1: Net-(U13-BOOT0) -> Net-(U22-BOOT0)
- SW1 pad 1: Net-(U13-BOOT0) -> Net-(U22-BOOT0)
- SW2 pad 1: /NRST -> GND
- SW2 pad 2: GND -> /NRST
- TP7 pad 1: Net-(U13-BOOT0) -> Net-(U22-BOOT0)
- TP8 pad 1: Net-(U13-PB2) -> Net-(U22-PB2)
- U7 pad 2: (no net) -> GND
- U7 pad 5: (no net) -> +5C
Other:
- board text removed: "Freewheel diodes"
