File: hw_v2/hw_v1.kicad_sch (KiCad schematic)
At the start: 54 parts, among them J16 47352-1001, J8 USB_B_Micro, J9 Tag connect, SW1 SW_Push, SW2 SW_Push, U14 TJA1051T-3, U15 25Q16, U16 REF3033, U17 SRV05-4, U22 STM32F407VGTx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

Commit message: wip routing iny/ign drivers
Parts:
- C32, C34: now not fitted; now left out of the parts list
Changed lines of the file:
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@@
 		(unit 1)
 		(exclude_from_sim no)
-		(in_bom yes)
-		(on_board yes)
-		(dnp no)
+		(in_bom no)
+		(on_board no)
+		(dnp yes)
 		(property "Reference" "C32"
 			(at 156.972 180.34 0)
@@
 		(unit 1)
 		(exclude_from_sim no)
-		(in_bom yes)
-		(on_board yes)
-		(dnp no)
+		(in_bom no)
+		(on_board no)
+		(dnp yes)
 		(property "Reference" "C34"
 			(at 168.91 182.88 0)

Commit message: wip mcu routing
Connections:
- net CEL_OUT: now also U22.93 (PB7); no longer U22.15 (PC0)
- net CLT: now also U22.23 (PA0); no longer U22.26 (PA3)
- net IAT: now also U22.26 (PA3); no longer U22.23 (PA0)
- net RPM_OUT: now also U22.92 (PB6); no longer U22.42 (PE11)
- net fan1: now also U22.2 (PE3); no longer U22.1 (PE2)
- net fan2: now also U22.1 (PE2); no longer U22.3 (PE4)
- net fuel_pump: now also U22.3 (PE4); no longer U22.2 (PE3)
- no-connect marks 25 -> 23
Other:
- note removed: "DEBUG PIN"
Changed lines of the file:
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@@
 		)
 	)
-	(text "DEBUG PIN"
-		(exclude_from_sim no)
-		(at 96.52 94.488 0)
-		(effects
-			(font
-				(size 0.889 0.889)
-			)
-			(justify left bottom)
-		)
-	)
 	(text "USB"
 		(exclude_from_sim no)
@@
 	)
 	(no_connect
-		(at 95.25 101.6)
-	)
-	(no_connect
 		(at 95.25 142.24)
 	)
@@
 	)
 	(no_connect
-		(at 95.25 99.06)
-	)
-	(no_connect
 		(at 179.07 52.07)
 	)
@@
 	(wire
 		(pts
+			(xy 95.25 99.06) (xy 97.79 99.06)
+		)
+		(stroke
+			(width 0)
+			(type default)
+		)
+	)
+	(wire
+		(pts
 			(xy 184.15 21.59) (xy 184.15 22.86)
 		)
@@
 	(wire
 		(pts
+			(xy 97.79 101.6) (xy 95.25 101.6)
+		)
+		(stroke
+			(width 0)
+			(type default)
+		)
+	)
+	(wire
+		(pts
 			(xy 171.45 110.49) (xy 171.45 111.76)
 		)
@@
 	)
 	(label "fuel_pump"
-		(at 35.56 71.12 0)
+		(at 35.56 73.66 0)
 		(effects
 			(font
@@
 	)
 	(label "IAT"
-		(at 102.87 40.64 180)
+		(at 102.87 48.26 180)
 		(effects
 			(font
@@
 	)
 	(label "RPM_OUT"
-		(at 35.56 91.44 0)
+		(at 97.79 99.06 0)
 		(effects
 			(font
@@
 	)
 	(label "fan1"
-		(at 35.56 68.58 0)
+		(at 35.56 71.12 0)
 		(effects
 			(font
@@
 	)
 	(label "CEL_OUT"
-		(at 104.14 127 180)
+		(at 97.79 101.6 0)
 		(effects
 			(font
 				(size 0.8 0.8)
 			)
-			(justify right bottom)
+			(justify left bottom)
 		)
 	)
 	(label "fan2"
-		(at 35.56 73.66 0)
+		(at 35.56 68.58 0)
 		(effects
 			(font
@@
 	)
 	(label "CLT"
-		(at 102.87 48.26 180)
+		(at 102.87 40.64 180)
 		(effects
 			(font

Commit message: update ADC oamp
Parts:
- RN3: LCSC (none) -> C102673
- U22: LCSC (none) -> C12345
Connections:
- net ACCL_CS: now also U22.35 (PB0); no longer U22.95 (PB8)
- net BARO_CS: now also U22.36 (PB1); no longer U22.96 (PB9)
- net ECN1: now also U22.62 (PD15); no longer U22.59 (PD12)
- net ECN2: now also U22.61 (PD14); no longer U22.60 (PD13)
- net ECN3: now also U22.56 (PD9); no longer U22.61 (PD14)
- net ECN4: now also U22.59 (PD12); no longer U22.62 (PD15)
- net INY1: now also U22.58 (PD11); no longer U22.55 (PD8)
- net INY2: now also U22.60 (PD13); no longer U22.56 (PD9)
- net INY3: now also U22.55 (PD8); no longer U22.57 (PD10)
- net INY4: now also U22.57 (PD10); no longer U22.58 (PD11)
- net MEMORY_CS: now also U22.34 (PC5); no longer U22.52 (PB13)
- net MTR_DIR: now also U22.40 (PE9); no longer U22.39 (PE8)
- net MTR_ENABLE: now also U22.38 (PE7); no longer U22.41 (PE10)
- net MTR_FAULT: now also U22.39 (PE8); no longer U22.40 (PE9)
- net MTR_STEP: now also U22.41 (PE10); no longer U22.38 (PE7)
- net SD_CARD_DETECT: now also U22.42 (PE11); no longer U22.66 (PC9)
- net SD_CS: now also U22.33 (PC4); no longer U22.65 (PC8), U22.83 (PD2)
- net SPI3_MISO: now also RN3.4 (R4.1); no longer RN3.3 (R3.1)
- net SPI3_SCk: now also RN3.3 (R3.1); no longer RN3.4 (R4.1)
- net SW_AC_m: now also U22.45 (PE14); no longer U22.43 (PE12)
- net SW_TABLE_m: now also U22.43 (PE12); no longer U22.45 (PE14)
- no-connect marks 23 -> 24
Changed lines of the file:
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@@
 	)
 	(no_connect
-		(at 95.25 137.16)
-	)
-	(no_connect
-		(at 95.25 86.36)
-	)
-	(no_connect
 		(at 95.25 93.98)
 	)
@@
 	)
 	(no_connect
+		(at 104.14 116.84)
+	)
+	(no_connect
 		(at 95.25 142.24)
 	)
@@
 	)
 	(no_connect
-		(at 95.25 83.82)
+		(at 95.25 96.52)
 	)
 	(no_connect
-		(at 95.25 96.52)
+		(at 96.52 106.68)
+	)
+	(no_connect
+		(at 35.56 111.76)
+	)
+	(no_connect
+		(at 97.79 104.14)
 	)
 	(no_connect
@@
 	)
 	(no_connect
+		(at 97.79 147.32)
+	)
+	(no_connect
 		(at 95.25 78.74)
 	)
@@
 		(at 95.25 111.76)
 	)
-	(no_connect
-		(at 95.25 139.7)
-	)
 	(wire
 		(pts
@@
 	)
 	(label "MTR_STEP"
-		(at 35.56 81.28 0)
+		(at 35.56 88.9 0)
 		(effects
 			(font
@@
 	)
 	(label "ECN4"
-		(at 35.56 144.78 0)
+		(at 35.56 137.16 0)
 		(effects
 			(font
@@
 	)
 	(label "INY4"
-		(at 35.56 134.62 0)
+		(at 35.56 132.08 0)
 		(effects
 			(font
@@
 	)
 	(label "MTR_FAULT"
-		(at 35.56 86.36 0)
+		(at 35.56 83.82 0)
 		(effects
 			(font
@@
 	)
 	(label "ECN1"
-		(at 35.56 137.16 0)
+		(at 35.56 144.78 0)
 		(effects
 			(font
@@
 	)
 	(label "SPI3_SCk"
-		(at 203.2 39.37 270)
+		(at 200.66 39.37 270)
 		(effects
 			(font
@@
 	)
 	(label "SW_TABLE_m"
-		(at 35.56 99.06 0)
+		(at 35.56 93.98 0)
 		(effects
 			(font
@@
 	)
 	(label "ECN3"
-		(at 35.56 142.24 0)
+		(at 35.56 129.54 0)
 		(effects
 			(font
@@
 		)
 	)
-	(label "SD_CS"
-		(at 97.79 147.32 0)
-		(effects
-			(font
-				(size 0.7874 0.7874)
-			)
-			(justify left bottom)
-		)
-	)
 	(label "VBATT"
 		(at 198.12 76.2 180)
@@
 	)
 	(label "ECN2"
-		(at 35.56 139.7 0)
+		(at 35.56 142.24 0)
 		(effects
 			(font
@@
 	)
 	(label "MTR_DIR"
-		(at 35.56 83.82 0)
+		(at 35.56 86.36 0)
 		(effects
 			(font
@@
 	)
 	(label "INY2"
-		(at 35.56 129.54 0)
+		(at 35.56 139.7 0)
 		(effects
 			(font
@@
 	)
 	(label "SD_CS"
-		(at 35.56 111.76 0)
+		(at 95.25 137.16 0)
 		(effects
 			(font
@@
 	)
 	(label "MEMORY_CS"
-		(at 104.14 116.84 180)
+		(at 95.25 139.7 0)
 		(effects
 			(font
 				(size 0.8 0.8)
 			)
-			(justify right bottom)
+			(justify left bottom)
 		)
 	)
@@
 	)
 	(label "INY3"
-		(at 35.56 132.08 0)
+		(at 35.56 127 0)
 		(effects
 			(font
@@
 	)
 	(label "MTR_ENABLE"
-		(at 35.56 88.9 0)
+		(at 35.56 81.28 0)
 		(effects
 			(font
@@
 	)
 	(label "SD_CARD_DETECT"
-		(at 97.79 149.86 0)
+		(at 35.56 91.44 0)
 		(effects
 			(font
@@
 	)
 	(label "INY1"
-		(at 35.56 127 0)
+		(at 35.56 134.62 0)
 		(effects
 			(font
@@
 	)
 	(label "SW_AC_m"
-		(at 35.56 93.98 0)
+		(at 35.56 99.06 0)
 		(effects
 			(font
@@
 	)
 	(label "SPI3_MISO"
-		(at 200.66 39.37 270)
+		(at 203.2 39.37 270)
 		(effects
 			(font
@@
 	(global_label "BARO_CS"
 		(shape input)
-		(at 97.79 106.68 0)
+		(at 95.25 86.36 0)
 		(fields_autoplaced yes)
 		(effects
@@
 		)
 		(property "Intersheetrefs" "${INTERSHEET_REFS}"
-			(at 104.9655 106.68 0)
+			(at 102.4255 86.36 0)
 			(effects
 				(font
@@
 	(global_label "ACCL_CS"
 		(shape input)
-		(at 97.79 104.14 0)
+		(at 95.25 83.82 0)
 		(fields_autoplaced yes)
 		(effects
@@
 		)
 		(property "Intersheetrefs" "${INTERSHEET_REFS}"
-			(at 104.775 104.14 0)
+			(at 102.235 83.82 0)
 			(effects
 				(font
@@
 			)
 		)
+		(property "LCSC" "C102673"
+			(at 205.74 33.0199 0)
+			(effects
+				(font
+					(size 1.27 1.27)
+				)
+				(hide yes)
+			)
+		)
 		(pin "6"
 		)
@@
 			(effects
 				(font
+					(size 1.27 1.27)
+				)
+				(hide yes)
+			)
+		)
+		(property "LCSC" "C12345"
+			(at 74.5333 172.72 0)
+			(effects
+				(font
