File: hw_v2/pmic.kicad_sch (KiCad schematic)
At the start: 17 parts, among them U2 TC4424A, U3 TC4424A

Commit message: WIP v7
Parts:
- added R5, R6, R8, R9: 4.7k, hellen-one-common:R0603, symbol hellen-one-common:Res
- added U12, U20: VNLD5160TR-E, Package_SO:SOIC-8_3.9x4.9mm_P1.27mm, symbol chips:VNLD5160
- JP13: now fitted
Connections:
- net ECN1: now also U2.2 (IN_A)
- net ECN2: now also U2.4 (IN_B)
- net ECN3: now also U3.2 (IN_A)
- net ECN4: now also U3.4 (IN_B)
- net GND: now also R5.1, R6.1, R8.1, R9.1, U12.5 (S2), U12.7 (S1), U20.5 (S2), U20.7 (S1)
- net INJ-1-OUT: now also U12.8 (D1)
- net INJ-2-OUT: now also U12.6 (D2)
- net INJ-3-OUT: now also U20.8 (D1)
- net INJ-4-OUT: now also U20.6 (D2)
- net INY1: now also R8.2, U12.1 (IN1); no longer U2.2 (IN_A)
- net INY2: now also R5.2, U12.3 (IN2); no longer U2.4 (IN_B)
- net INY3: now also R9.2, U20.1 (IN1); no longer U3.2 (IN_A)
- net INY4: now also R6.2, U20.3 (IN2); no longer U3.4 (IN_B)
- no-connect marks 0 -> 4
Other:
- moved on the sheet: U2, U3

Commit message: hw v2
Parts:
- R5, R6, R8, R9: footprint hellen-one-common:R0603 -> Resistor_SMD:R_0603_1608Metric
Changed lines of the file:
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@@
 			)
 		)
-		(property "Footprint" "hellen-one-common:R0603"
+		(property "Footprint" "Resistor_SMD:R_0603_1608Metric"
 			(at 142.24 135.89 0)
 			(effects
@@
 			)
 		)
-		(property "Footprint" "hellen-one-common:R0603"
+		(property "Footprint" "Resistor_SMD:R_0603_1608Metric"
 			(at 154.94 104.14 0)
 			(effects
@@
 			)
 		)
-		(property "Footprint" "hellen-one-common:R0603"
+		(property "Footprint" "Resistor_SMD:R_0603_1608Metric"
 			(at 154.94 130.81 0)
 			(effects
@@
 			)
 		)
-		(property "Footprint" "hellen-one-common:R0603"
+		(property "Footprint" "Resistor_SMD:R_0603_1608Metric"
 			(at 140.97 109.22 0)
 			(effects

Commit message: wip analog frontend & power
Connections:
- net IGN-1-OUT: now also RN1.4 (R4.1); no longer RN1.5 (R4.2)
- net IGN-2-OUT: now also RN1.3 (R3.1); no longer RN1.6 (R3.2)
- net IGN-3-OUT: now also RN1.2 (R2.1); no longer RN1.7 (R2.2)
- net IGN-4-OUT: now also RN1.1 (R1.1); no longer RN1.8 (R1.2)
- net at D1.2 (A): now also RN1.8 (R1.2); no longer RN1.1 (R1.1)
- net at D12.2 (A): now also RN1.5 (R4.2); no longer RN1.4 (R4.1)
- net at D4.2 (A): now also RN1.7 (R2.2); no longer RN1.2 (R2.1)
- net at D9.2 (A): now also RN1.6 (R3.2); no longer RN1.3 (R3.1)
Other:
- moved on the sheet: RN1
Changed lines of the file:
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@@
 	(symbol
 		(lib_id "Device:R_Pack04")
-		(at 233.68 80.01 90)
+		(at 233.68 80.01 270)
+		(mirror x)
 		(unit 1)
 		(exclude_from_sim no)
@@
 		(on_board yes)
 		(dnp no)
-		(fields_autoplaced yes)
 		(property "Reference" "RN1"
-			(at 232.41 74.93 0)
+			(at 233.68 91.44 90)
 			(effects
 				(font
 					(size 1.27 1.27)
 				)
-				(justify left)
 			)
 		)
 		(property "Value" "1k"
-			(at 234.95 74.93 0)
+			(at 233.68 88.9 90)
 			(effects
 				(font
 					(size 1.27 1.27)
 				)
-				(justify left)
 			)
 		)

Commit message: planito mas catolico
Parts:
- removed R5, R6, R8, R9: 4.7k, Resistor_SMD:R_0603_1608Metric, symbol hellen-one-common:Res
- removed U12, U20: VNLD5160TR-E, Package_SO:SOIC-8_3.9x4.9mm_P1.27mm, symbol chips:VNLD5160
- removed U2, U3: TC4424A, Package_SO:SOIC-8_3.9x4.9mm_P1.27mm, symbol IC_Automotive:TC4424A
- added R12, R13, R14, R15, R5, R6, R8, R9: 4.7K, symbol Device:R_Small
- added U13, U20: ~, symbol hw_v2:VNLD5160TR-E
- added U2, U3: ~, symbol hw_v2:TC4424A
Connections:
- net ECN1: now also R12.1, U2.2 (IN_A)
- net ECN2: now also R13.1, U2.4 (IN_B)
- net ECN3: now also R14.1, U3.2 (IN_A)
- net ECN4: now also R15.1, U3.4 (IN_B)
- net GND: now also R12.2, R13.2, R14.2, R15.2, R5.2, R6.2, R8.2, R9.2, U13.5 (S2), U13.7 (S1), U2.3 (GND), U20.5 (S2), U20.7 (S1), U3.3 (GND)
- net IGN-1-OUT: now also U2.7 (OUT_A)
- net IGN-2-OUT: now also U2.5 (OUT_B)
- net IGN-3-OUT: now also U3.7 (OUT_A)
- net IGN-4-OUT: now also U3.5 (OUT_B)
- net IGN_V+: now also U2.6 (VDD), U3.6 (VDD)
- net INJ-1-OUT: now also U13.8 (D1)
- net INJ-2-OUT: now also U13.6 (D2)
- net INJ-3-OUT: now also U20.8 (D1)
- net INJ-4-OUT: now also U20.6 (D2)
- net INY1: now also R9.1, U13.1 (IN1)
- net INY2: now also R8.1, U13.3 (IN2)
- net INY3: now also R6.1, U20.1 (IN1)
- net INY4: now also R5.1, U20.3 (IN2)

Commit message: wip CKP/CMP
Parts:
- R12, R13, R14, R15, R5, R6, R8, R9: footprint (none) -> Resistor_SMD:R_0603_1608Metric
- U13, U20: footprint (none) -> Package_SO:SO-8_3.9x4.9mm_P1.27mm
- U2, U3: footprint (none) -> Package_SO:SOIC-8_3.9x4.9mm_P1.27mm
Changed lines of the file:
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@@
 (kicad_sch
-	(version 20241004)
+	(version 20241209)
 	(generator "eeschema")
 	(generator_version "8.99")
@@
 			)
 		)
-		(property "Footprint" ""
+		(property "Footprint" "Resistor_SMD:R_0603_1608Metric"
 			(at 87.63 132.08 0)
 			(effects
@@
 			)
 		)
-		(property "Footprint" ""
+		(property "Footprint" "Resistor_SMD:R_0603_1608Metric"
 			(at 100.33 135.89 0)
 			(effects
@@
 			)
 		)
-		(property "Footprint" ""
+		(property "Footprint" "Package_SO:SOIC-8_3.9x4.9mm_P1.27mm"
 			(at 116.84 68.58 0)
 			(effects
@@
 			)
 		)
-		(property "Footprint" ""
+		(property "Footprint" "Resistor_SMD:R_0603_1608Metric"
 			(at 90.17 86.36 0)
 			(effects
@@
 			)
 		)
-		(property "Footprint" ""
+		(property "Footprint" "Resistor_SMD:R_0603_1608Metric"
 			(at 87.63 109.22 0)
 			(effects
@@
 			)
 		)
-		(property "Footprint" ""
+		(property "Footprint" "Resistor_SMD:R_0603_1608Metric"
 			(at 92.71 86.36 0)
 			(effects
@@
 			)
 		)
-		(property "Footprint" ""
+		(property "Footprint" "Package_SO:SOIC-8_3.9x4.9mm_P1.27mm"
 			(at 116.84 52.07 0)
 			(effects
@@
 			)
 		)
-		(property "Footprint" ""
+		(property "Footprint" "Resistor_SMD:R_0603_1608Metric"
 			(at 100.33 113.03 0)
 			(effects
@@
 			)
 		)
-		(property "Footprint" ""
+		(property "Footprint" "Resistor_SMD:R_0603_1608Metric"
 			(at 95.25 86.36 0)
 			(effects
@@
 			)
 		)
-		(property "Footprint" ""
+		(property "Footprint" "Package_SO:SO-8_3.9x4.9mm_P1.27mm"
 			(at 115.57 105.41 0)
 			(effects
@@
 			)
 		)
-		(property "Footprint" ""
+		(property "Footprint" "Resistor_SMD:R_0603_1608Metric"
 			(at 97.79 86.36 0)
 			(effects
@@
 			)
 		)
-		(property "Footprint" ""
+		(property "Footprint" "Package_SO:SO-8_3.9x4.9mm_P1.27mm"
 			(at 115.57 128.27 0)
 			(effects
