File: hw_v2/protoboard.kicad_sch (KiCad schematic)
At the start: 17 parts, among them J15 Conn_01x03, J2 Conn_01x05, J3 Conn_01x05, J4 Conn_01x05, J5 Conn_01x03, J6 Conn_01x04

Commit message: fix LCSC codes
Parts:
- C19, C25: LCSC C49678 -> C1525
- D16: LCSC C191023 -> C85364
- D17: LCSC C191023 -> C22452
- R16: LCSC C21190 -> C13167
Changed lines of the file:
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@@
 			)
 		)
-		(property "LCSC" "C49678"
+		(property "LCSC" "C1525"
 			(at 148.59 68.58 0)
 			(effects
@@
 			)
 		)
-		(property "LCSC" "C191023"
+		(property "LCSC" "C22452"
 			(at 137.16 46.99 0)
 			(effects
@@
 			)
 		)
-		(property "LCSC" "C21190"
+		(property "LCSC" "C13167"
 			(at 167.64 46.99 90)
 			(effects
@@
 			)
 		)
-		(property "LCSC" "C49678"
+		(property "LCSC" "C1525"
 			(at 167.64 73.66 0)
 			(effects
@@
 			)
 		)
-		(property "LCSC" "C191023"
+		(property "LCSC" "C85364"
 			(at 148.59 45.72 0)
 			(effects

Commit message: update ADC oamp
Parts:
- R12, R13: LCSC C114564 -> C23162
Changed lines of the file:
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@@
 			)
 		)
-		(property "LCSC" "C114564"
+		(property "LCSC" "C23162"
 			(at 130.81 59.69 0)
 			(effects
@@
 			)
 		)
-		(property "LCSC" "C114564"
+		(property "LCSC" "C23162"
 			(at 130.81 57.15 0)
 			(effects
